File: Kicad/DebugAndOtherPeripheralsBoard/DebugAndOtherPeripheralsBoard.kicad_sch (KiCad schematic)
At the start: 118 parts, among them J1 SCL, SDA, +, GND, J10 USB RWGBS, J11 Standoff Hole, J12 Standoff Hole, J13 Standoff Hole, J14 Standoff Hole, J15 Standoff Hole, J2 Conn_01x08_Pin, J3 Conn_01x01_Pin, J4 Conn_01x01_Pin, J5 +36V, J6 GND, J7 Conn_01x04_Pin, J8 Conn_01x04_Pin, J9 USB RWGBS

Commit message: ProgrammingHelper
Utility that has buttons to quickly spin up the console if not open and send commands for configuring building flashing monitoring. This automatically establishes the com port to avoid confusion by myself and potentially flashing the wrong code to the wrong device. Much quicker and cleaner.
Parts:
- removed C1: C_drive 1uF, Custom:C320C105K5R5TA, symbol Device:C
- removed C17, C45: ~, Capacitor_THT:C_Rect_L7.0mm_W2.5mm_P5.00mm, symbol Custom:C317C300J5G5TA
- removed C18, C27, C46: ~, Capacitor_THT:C_Rect_L7.0mm_W2.5mm_P5.00mm, symbol Custom:C322C104J5R5TA
- removed C19: 0.1uF within 2mm, Capacitor_THT:C_Disc_D7.0mm_W2.5mm_P5.00mm, symbol Device:C
- removed C20, C21, C22, C23, C29, C30, C31, C32, C33, C34, C35, C36, C37, C38, C39, C40, C41, C42, C43, C44: EKYB101ELL102MM40S, Custom:EKYB101ELL102MM40S, symbol Device:C_Polarized
- removed C24: 0.1uF low ESR Ceramic, Capacitor_THT:C_Rect_L7.0mm_W2.5mm_P5.00mm, symbol Device:C
- removed C25: 100uF UHD1H101MPD1TD, Custom:UHD1H101MPD1TD, symbol Device:C
- removed C28: 1uF, Custom:C320C105K5R5TA, symbol Device:C
- removed C47, C48, C49, C50, C51, C52: R75RR322050L4J, Custom:R75RR322050L4J, symbol Device:C
- removed D1, D8: MBR40250G, Custom:MBR40250G, symbol Device:D
- removed D2, D3: ~, Diode_THT:D_DO-35_SOD27_P7.62mm_Horizontal, symbol Custom:1N4619
- removed D5, D6: 1N4148, Diode_THT:D_DO-35_SOD27_P7.62mm_Horizontal, symbol Diode:1N4148
- removed H1: Heatsink 1, Custom:647-25ABEP, symbol Connector:Conn_01x01_Pin
- removed H2: Heatsink 2, Custom:647-25ABEP, symbol Connector:Conn_01x01_Pin
- removed H5: Heatsink 5, Custom:647-25ABEP, symbol Connector:Conn_01x01_Pin
- removed J15: Standoff Hole, Custom:ContactViaM3, symbol Connector:Conn_01x01_Pin
- removed J3, J4: Conn_01x01_Pin, Custom:5055556-9, symbol Connector:Conn_01x01_Pin
- removed L1: SER2918H-223KL, Custom:SER2918H-223KL, symbol Device:L
- removed L2: 74436411500, Custom:74436411500, symbol Device:L
- removed OR6, OR7: ~, Custom:RS PRO Optical Receiver jack, symbol Custom:RS_PRO_Optical_Receiver_jack
- removed OT4: ~, Custom:RS Pro Optical Transmitter jack, symbol Custom:RS_PRO_Optical_Transmitter_Jack
- removed R12: R_pfb_i 1K, Resistor_THT:R_Axial_DIN0207_L6.3mm_D2.5mm_P7.62mm_Horizontal, symbol Device:R
- removed R13: R_sfb_i 1K, Resistor_THT:R_Axial_DIN0207_L6.3mm_D2.5mm_P7.62mm_Horizontal, symbol Device:R
- removed R14: R_pulldown 1000, Resistor_THT:R_Axial_DIN0207_L6.3mm_D2.5mm_P7.62mm_Horizontal, symbol Device:R_Small
- removed R15: 3K, Resistor_THT:R_Axial_DIN0207_L6.3mm_D2.5mm_P7.62mm_Horizontal, symbol Device:R
- removed R17: 1.33K, Resistor_THT:R_Axial_DIN0309_L9.0mm_D3.2mm_P12.70mm_Horizontal, symbol Device:R
- removed R4: ~, Custom:RX24-100W, symbol Custom:RX24-100W
- removed R9: R_pcfb_sense 0.001, Custom:PCS2512FR0010ET, symbol Device:R
- removed U1: ~, Package_DIP:CERDIP-8_W7.62mm_SideBrazed_LongPads, symbol Custom:TC1413N
- removed U2: ~, Package_DIP:CERDIP-8_W7.62mm_SideBrazed_LongPads, symbol Custom:MCP6021-E/P
- removed U3: ~, Package_TO_SOT_THT:TO-92, symbol Custom:LM4040C25ILPR
- removed U4: ~, Custom:IXFP60N25X3, symbol Custom:IXFP60N25X3
- added C1: 1000uF UPW1E102MHD, Custom:UPW1E102MHD, symbol Device:C_Polarized
- added D1, D2, D3: 1N4148, Diode_THT:D_DO-35_SOD27_P7.62mm_Horizontal, symbol Diode:1N4148
- added J15, J16, J17, J3, J4: Conn_01x04_Pin, TerminalBlock:TerminalBlock_MaiXu_MX126-5.0-04P_1x04_P5.00mm, symbol Connector:Conn_01x04_Pin
- added R4, R9: 10K, Resistor_THT:R_Axial_DIN0207_L6.3mm_D2.5mm_P7.62mm_Horizontal, symbol Device:R_Small
- added U1, U3: ~, Custom:AWHSH124D00G, symbol Custom:AWHSH124D00G
- added U2, U4, U8: ~, Package_TO_SOT_THT:TO-92, symbol Custom:2N7000
- R1: value R_drive 5 -> 10K; footprint Resistor_THT:R_Axial_DIN0207_L6.3mm_D2.5mm_P10.16mm_Horizontal -> Resistor_THT:R_Axial_DIN0207_L6.3mm_D2.5mm_P7.62mm_Horizontal
- R10: value R_pcfb_in 1K -> 1K
- R11: value R_pcfb_f 56K -> 1.33K; footprint Resistor_THT:R_Axial_DIN0207_L6.3mm_D2.5mm_P7.62mm_Horizontal -> Resistor_THT:R_Axial_DIN0309_L9.0mm_D3.2mm_P12.70mm_Horizontal
- R2: value R_sfb_H 500K -> 1K
- R3: value R_sfb_L 6.8K -> 1.33K; footprint Resistor_THT:R_Axial_DIN0207_L6.3mm_D2.5mm_P7.62mm_Horizontal -> Resistor_THT:R_Axial_DIN0309_L9.0mm_D3.2mm_P12.70mm_Horizontal
- R7: value R_pfb_H 270K -> 1K
- R8: value R_pfb_ 10K -> 1.33K; footprint Resistor_THT:R_Axial_DIN0207_L6.3mm_D2.5mm_P7.62mm_Horizontal -> Resistor_THT:R_Axial_DIN0309_L9.0mm_D3.2mm_P12.70mm_Horizontal
Connections:
- net +3V3: now also J15.2 (Pin_2), J16.2 (Pin_2), J17.4 (Pin_4), J3.2 (Pin_2), J4.2 (Pin_2); no longer J7.4 (Pin_4)
- net Earth: now also R1.2, U6.4, U7.4, C1.2, J17.1 (Pin_1), J17.2 (Pin_2), R4.2, R9.2, U1.4, U2.1 (S), U3.4, U4.1 (S), U8.1 (S); no longer R10.2, R3.2, R8.2, U7.1
- net at R8.1: now also D2.2 (A), U3.1; no longer R7.2
- net at R7.1: now also X1.10 (D27_a2io), R4.1
- net at X1.11 (D14_a2io): now also R1.1, R2.1
- net at R3.1: now also D1.2 (A), U1.1; no longer R2.2
- net +12V: now reaches U7.3
- net +12V: now also D4.1 (K), J8.4 (Pin_4), U6.3, C1.1, D1.1 (K), D2.1 (K), D3.1 (K), J15.4 (Pin_4), J16.4 (Pin_4), J3.4 (Pin_4), J4.4 (Pin_4), U1.3, U3.3
- net at R11.2: now also U8.3 (D); no longer R10.1
- net at R11.1: now also U7.1, D3.2 (A); no longer X1.4 (D34_a1i)
- net at U7.2: now also J16.1 (Pin_1); no longer F1.2
- net at X1.9 (D26_a2io): now also R10.1, R9.1
- net +10V renamed +5V
- net +5V: now also J7.4 (Pin_4), J15.3 (Pin_3), J16.3 (Pin_3), J3.3 (Pin_3), J4.3 (Pin_3); no longer J8.4 (Pin_4)
- new net: J4.1 (Pin_1), U1.2
- new net: F1.2, J17.3 (Pin_3), J7.3 (Pin_3), J8.3 (Pin_3)
- new net: R2.2, U2.2 (G)
- new net: J3.1 (Pin_1), U6.2
- new net: R7.2, U4.2 (G)
- new net: R10.2, U8.2 (G)
- new net: R3.2, U2.3 (D)
- new net: R8.2, U4.3 (D)
- new net: J15.1 (Pin_1), U3.2
Other:
- note removed: "2.5V Reference"
- note removed: "Driver"
- note removed: "First Stage Voltage Feedback"
- note removed: "Flyback Connections"
- note removed: "High Power Supply Voltage Feedback"
- note removed: "Optical Peripherals Interface"
- note removed: "Output Current Feedback"
- note removed: "Output Voltage Feedback"
- note removed: "Power Conditioning"
- note removed: "Primary Current Feedback"
- note removed: "Snubber"
- note removed: "Snubber Voltage Feedback"
- moved on the sheet: C2, C3, D4, F1, J11, J12, J13, J14, J5, J6, J7, J8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
