File: Kicad/HVPSController/HVPSController.kicad_sch (KiCad schematic)
At the start: 118 parts, among them J1 SCL, SDA, +, GND, J10 USB RWGBS, J11 Standoff Hole, J12 Standoff Hole, J13 Standoff Hole, J14 Standoff Hole, J15 Standoff Hole, J2 Conn_01x08_Pin, J3 Conn_01x01_Pin, J4 Conn_01x01_Pin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

Commit message: Putting temperature sensing in place.
Parts:
- J1: value SCL, SDA, +, GND -> SCL, SDA, GND, +
Changed lines of the file:
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@@
 			)
 		)
-		(property "Value" "SCL, SDA, +, GND"
+		(property "Value" "SCL, SDA, GND, +"
 			(at 116.84 269.24 90)
 			(effects

Commit message: having a hard time pulling myself away from this. Must stop now.
Parts:
- D5: footprint Diode_THT:D_DO-35_SOD27_P7.62mm_Horizontal -> Diode_THT:D_DO-35_SOD27_P5.08mm_Vertical_AnodeUp
Changed lines of the file:
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@@
 			)
 		)
-		(property "Footprint" "Diode_THT:D_DO-35_SOD27_P7.62mm_Horizontal"
+		(property "Footprint" "Diode_THT:D_DO-35_SOD27_P5.08mm_Vertical_AnodeUp"
 			(at 364.49 172.72 0)
 			(effects
