File: Kicad/HVPSController2/HVPSController2.kicad_pcb (KiCad board)
At the start: 2 copper layers, 234.5 x 198.2 mm, 118 parts, among them J1 SCL, SDA, +, GND, J10 USB RWGBS, J11 Standoff Hole, J12 Standoff Hole, J13 Standoff Hole, J14 Standoff Hole, J15 Standoff Hole, J2 Conn_01x08_Pin, J3 Conn_01x01_Pin, J4 Conn_01x01_Pin, J5 +36V, J6 GND, J7 Conn_01x04_Pin, J8 Conn_01x04_Pin, J9 USB RWGBS

Commit message: having a hard time pulling myself away from this. Must stop now.
Parts:
- removed C39: EKYB101ELL102MM40S, Custom:EKYB101ELL102MM40S
- removed H5: Heatsink 5, Custom:647-25ABEP
- removed J7: Conn_01x04_Pin, TerminalBlock:TerminalBlock_MaiXu_MX126-5.0-04P_1x04_P5.00mm
- removed OR7: ~, Custom:RS PRO Optical Receiver jack
- removed X1: ~, Custom:ESP32_WROOM-32_Dev_Board
- added C26: ~, Capacitor_THT:C_Rect_L7.0mm_W2.5mm_P5.00mm, F.Cu at (304.6, 23.2)
- added C53: C, Capacitor_THT:C_Rect_L7.0mm_W2.5mm_P5.00mm, F.Cu at (160.4, 23.3)
- added C54: 0.1uF, Capacitor_THT:C_Rect_L7.0mm_W2.5mm_P5.00mm, F.Cu at (124.3, -22.8)
- added C55: 0.1uF, Capacitor_THT:C_Rect_L7.0mm_W2.5mm_P5.00mm, F.Cu at (124.3, -18.7)
- added C56: 10uF, Capacitor_THT:C_Rect_L4.0mm_W2.5mm_P2.50mm, F.Cu at (146.0, -104.4)
- added C57: 2.2nF, Capacitor_THT:C_Rect_L7.0mm_W2.5mm_P5.00mm, F.Cu at (124.3, -14.7)
- added C58: 1000uF, Custom:ECA-1JM102, F.Cu at (246.6, 235.9)
- added C59: 0.1uF, Capacitor_THT:C_Rect_L7.0mm_W2.5mm_P5.00mm, F.Cu at (235.8, 236.2)
- added C62: 470uF, Custom:UPW1E471MPD6TA, F.Cu at (214.8, 226.7)
- added C63: 0.1uF, Capacitor_THT:C_Rect_L7.0mm_W2.5mm_P5.00mm, F.Cu at (212.8, 233.2)
- added C64: 0.1uF, Capacitor_THT:C_Rect_L7.0mm_W2.5mm_P5.00mm, F.Cu at (124.3, -2.51)
- added C65: 0.1uF, Capacitor_THT:C_Rect_L7.0mm_W2.5mm_P5.00mm, F.Cu at (124.3, 1.54)
- added C66: 10uF, Capacitor_THT:C_Rect_L4.0mm_W2.5mm_P2.50mm, F.Cu at (146.0, -100.3)
- added C67: 1uF FG26X7R2A105KNT06, Capacitor_THT:C_Rect_L7.0mm_W2.0mm_P5.00mm, F.Cu at (223.4, 122.7)
- added C68: FG26X7R2A105KNT06, Capacitor_THT:C_Rect_L7.0mm_W2.0mm_P5.00mm, F.Cu at (223.8, 205.6)
- added C69: 0.1uF, Capacitor_THT:C_Rect_L7.0mm_W2.5mm_P5.00mm, F.Cu at (124.3, 5.59)
- added C70: 10uF, Capacitor_THT:C_Rect_L4.0mm_W2.5mm_P2.50mm, F.Cu at (176.1, -22.8)
- added C71: 0.1uF, Capacitor_THT:C_Rect_L7.0mm_W2.5mm_P5.00mm, F.Cu at (124.3, 9.64)
- added C72: 10uF, Capacitor_THT:C_Rect_L4.0mm_W2.5mm_P2.50mm, F.Cu at (176.1, -18.7)
- added C73: 1uF, Capacitor_THT:C_Rect_L7.0mm_W2.0mm_P5.00mm, F.Cu at (215.4, 122.7)
- added C74: 1uF, Capacitor_THT:C_Rect_L7.0mm_W2.0mm_P5.00mm, F.Cu at (216.4, 205.6)
- added D10: 1N5822, Diode_THT:D_DO-201AD_P12.70mm_Horizontal, F.Cu at (461.2, 155.5)
- added D11: 1N4149, Diode_THT:D_DO-35_SOD27_P10.16mm_Horizontal, F.Cu at (206.5, 159.6)
- added D12: 1N4149, Diode_THT:D_DO-35_SOD27_P10.16mm_Horizontal, F.Cu at (215.0, 57.8)
- added D13: 1N5822, Diode_THT:D_DO-201AD_P12.70mm_Horizontal, F.Cu at (231.2, 237.8)
- added D14: MUR220RLG, Diode_THT:D_DO-41_SOD81_P7.62mm_Horizontal, B.Cu at (229.5, 115.9)
- added D15: MUR420 R0, Diode_THT:D_DO-41_SOD81_P7.62mm_Horizontal, F.Cu at (229.9, 211.7)
- added D16: 1N4148, Diode_THT:D_DO-35_SOD27_P10.16mm_Horizontal, F.Cu at (215.0, 61.3)
- added D7: 1N4149, Diode_THT:D_DO-35_SOD27_P10.16mm_Horizontal, F.Cu at (196.6, 171.3)
- added D9: 1N4149, Diode_THT:D_DO-35_SOD27_P10.16mm_Horizontal, F.Cu at (206.7, 167.3)
- added H3: Heatsink, Custom:647-25ABEP, F.Cu at (208.6, 139.2)
- added H4: Heatsink, Custom:647-25ABEP, F.Cu at (208.7, 190.0)
- added J11: USB RWGBS, Custom:USB connection, F.Cu at (228.7, 35.9)
- added J12: USB RWGBS, Custom:USB connection, F.Cu at (228.7, 42.1)
- added J13: Conn_01x01_Pin, Custom:PCB-3 (M4), F.Cu at (234.0, 160.5)
- added J16: Tap debug pin, Connector_PinHeader_2.54mm:PinHeader_1x01_P2.54mm_Vertical, F.Cu at (249.6, 50.1)
- added J17: Conn_01x02_Pin, Connector_JST:JST_XH_B2B-XH-A_1x02_P2.50mm_Vertical, F.Cu at (84.0, 205.2)
- added J18: ~, Connector_PinHeader_2.54mm:PinHeader_1x01_P2.54mm_Vertical, F.Cu at (376.5, 17.1)
- added J19: ~, Connector_PinHeader_2.54mm:PinHeader_1x01_P2.54mm_Vertical, F.Cu at (376.5, 25.6)
- added J21: Standoff Hole, Custom:ContactViaM3, F.Cu at (212.6, 28.5)
- added J24: Standoff Hole, Custom:ContactViaM3, F.Cu at (376.5, 34.1)
- added J25: Standoff Hole, Custom:ContactViaM3, F.Cu at (212.6, 37.0)
- added J26: Standoff Hole, Custom:ContactViaM3, F.Cu at (376.5, 42.6)
- added K1: ~, Custom:AWHSH124D00G, F.Cu at (282.4, 99.0)
- added K2: ~, Custom:AWHSH124D00G, F.Cu at (259.6, 97.1)
- added K3: ~, Custom:SRD-5VDC-SL-C, F.Cu at (90.0, 190.3)
- added L3: 68uH, Custom:5026 Inductor, F.Cu at (450.8, 150.0)
- added L4: 68uH, Custom:5026 Inductor, F.Cu at (220.8, 230.7)
- added L5: ~, Custom:5026 Inductor, F.Cu at (402.6, 154.6)
- added L6: ~, Custom:5026 Inductor, F.Cu at (412.1, 154.6)
- added L7: ~, Custom:5026 Inductor, F.Cu at (421.8, 154.6)
- added OT5: ~, Custom:RS Pro Optical Transmitter jack, F.Cu at (190.0, 82.8)
- added R20: 2K 1%, Resistor_THT:R_Axial_DIN0207_L6.3mm_D2.5mm_P7.62mm_Horizontal, F.Cu at (217.8, 243.7)
- added R21: 6.2, Resistor_THT:R_Axial_DIN0207_L6.3mm_D2.5mm_P7.62mm_Horizontal, F.Cu at (231.5, 122.6)
- added R22: 6.2, Resistor_THT:R_Axial_DIN0207_L6.3mm_D2.5mm_P10.16mm_Horizontal, F.Cu at (232.6, 205.8)
- added R23: 1000, Resistor_THT:R_Axial_DIN0207_L6.3mm_D2.5mm_P5.08mm_Vertical, F.Cu at (233.7, 129.6)
- added R24: 1000, Resistor_THT:R_Axial_DIN0207_L6.3mm_D2.5mm_P5.08mm_Vertical, F.Cu at (235.3, 195.1)
- added R27: 22K, Resistor_THT:R_Axial_DIN0207_L6.3mm_D2.5mm_P7.62mm_Horizontal, F.Cu at (124.1, -104.4)
- added R28: 1K, Resistor_THT:R_Axial_DIN0207_L6.3mm_D2.5mm_P7.62mm_Horizontal, F.Cu at (124.1, -100.3)
- added R29: 10K, Resistor_THT:R_Axial_DIN0207_L6.3mm_D2.5mm_P7.62mm_Horizontal, F.Cu at (154.2, -22.8)
- added R30: 6.2, Resistor_THT:R_Axial_DIN0207_L6.3mm_D2.5mm_P7.62mm_Horizontal, F.Cu at (212.5, 122.4)
- added R31: 6.2, Resistor_THT:R_Axial_DIN0207_L6.3mm_D2.5mm_P7.62mm_Horizontal, F.Cu at (212.3, 205.6)
- added R34: 1000, Resistor_THT:R_Axial_DIN0207_L6.3mm_D2.5mm_P7.62mm_Horizontal, F.Cu at (208.5, 130.0)
- added R35: 1000, Resistor_THT:R_Axial_DIN0207_L6.3mm_D2.5mm_P7.62mm_Horizontal, F.Cu at (205.2, 200.3)
- added R36: 4.7, Resistor_THT:R_Axial_DIN0207_L6.3mm_D2.5mm_P5.08mm_Vertical, B.Cu at (214.3, 115.9)
- added R37: 4.7, Resistor_THT:R_Axial_DIN0207_L6.3mm_D2.5mm_P5.08mm_Vertical, F.Cu at (214.8, 211.7)
- added RV1: 5K, Potentiometer_THT:Potentiometer_Bourns_3296W_Vertical, F.Cu at (442.8, 128.5)
- added RV2: 10K, Potentiometer_THT:Potentiometer_Bourns_3296W_Vertical, F.Cu at (442.8, 157.2)
- added RV3: 30K, Potentiometer_THT:Potentiometer_Bourns_3296W_Vertical, F.Cu at (212.8, 237.9)
- added RV4: 10K (adjust to 5K), Potentiometer_THT:Potentiometer_Bourns_3296W_Vertical, F.Cu at (277.1, 35.8)
- added RV5: 5K (adjusted to 1.38 for 23.8K total, Potentiometer_THT:Potentiometer_Bourns_3296W_Vertical, F.Cu at (277.1, 42.2)
- added S2: ~, Custom:SLW-1678105-6A-N-D, F.Cu at (64.0, 113.5)
- added T1: ~, Custom:CST2020-200L, F.Cu at (220.9, 164.6)
- added U10: ~, LED_THT:LED_D5.0mm-4_RGB_Wide_Pins, F.Cu at (74.7, 193.6)
- added U11: ~, LED_THT:LED_D5.0mm-4_RGB_Wide_Pins, F.Cu at (74.7, 184.6)
- added U12: ~, Package_DIP:DIP-20_W7.62mm_Socket_LongPads, F.Cu at (158.0, 191.8)
- added U13: ~, LED_THT:LED_D5.0mm-4_RGB_Wide_Pins, F.Cu at (67.2, 178.2)
- added U14: ~, LED_THT:LED_D5.0mm-4_RGB_Wide_Pins, F.Cu at (67.2, 187.2)
- added U15: ~, LED_THT:LED_D5.0mm-4_RGB_Wide_Pins, F.Cu at (67.2, 196.4)
- added U16: ~, LED_THT:LED_D5.0mm-4_RGB_Wide_Pins, F.Cu at (67.2, 205.7)
- added U17: ~, Custom:EP4CE6E22C8N_FPGA_Development_Board_, F.Cu at (141.0, 147.3)
- added U18: ~, Package_TO_SOT_THT:TO-92, F.Cu at (389.3, -4.63)
- added U19: ~, Package_TO_SOT_THT:TO-220-5_Vertical, F.Cu at (235.0, 241.4)
- added U20: ~, Package_DIP:DIP-20_W7.62mm_Socket_LongPads, F.Cu at (133.9, 191.8)
- added U21: ~, Custom:IXFP60N25X3_2, F.Cu at (243.2, 129.9)
- added U22: ~, Custom:IXFP60N25X3_2, F.Cu at (243.2, 199.3)
- added U23: ~, Package_DIP:DIP-14_W7.62mm_Socket_LongPads, F.Cu at (214.3, 119.7)
- added U24: ~, Package_DIP:DIP-14_W7.62mm_Socket_LongPads, B.Cu at (214.9, 208.0)
- added U25: ~, Package_TO_SOT_THT:TO-92, F.Cu at (401.8, 40.4)
- added U26: ~, Custom:IXFP60N25X3_2, F.Cu at (208.7, 135.2)
- added U27: ~, Custom:IXFP60N25X3_2, F.Cu at (208.7, 194.0)
- added U8: ~, LED_THT:LED_D5.0mm-4_RGB_Wide_Pins, F.Cu at (74.7, 212.1)
- added U9: ~, LED_THT:LED_D5.0mm-4_RGB_Wide_Pins, F.Cu at (74.7, 202.9)
- C1: value C_drive 1uF -> EKYB101ELL102MM40S; footprint Custom:C320C105K5R5TA -> Custom:EKYB101ELL102MM40S
- C10, C4, C5, C6, C7, C8, C9: value ~ -> EKYB101ELL102MM40S; footprint Capacitor_THT:C_Rect_L7.0mm_W2.5mm_P5.00mm -> Custom:EKYB101ELL102MM40S
- C19: value 0.1uF within 2mm -> ~; footprint Capacitor_THT:C_Disc_D7.0mm_W2.5mm_P5.00mm -> Capacitor_THT:C_Rect_L7.0mm_W2.5mm_P5.00mm
- C2, C3: value 1000uF UPW1E102MHD -> EKYB101ELL102MM40S; footprint Custom:UPW1E102MHD -> Custom:EKYB101ELL102MM40S
- C20, C21, C22, C23: value EKYB101ELL102MM40S -> ~; footprint Custom:EKYB101ELL102MM40S -> Capacitor_THT:C_Rect_L7.0mm_W2.5mm_P5.00mm
- C24: value 0.1uF low ESR Ceramic -> ~
- C25: value 100uF UHD1H101MPD1TD -> ~; footprint Custom:UHD1H101MPD1TD -> Capacitor_THT:C_Rect_L7.0mm_W2.5mm_P5.00mm
- C28: value 1uF -> EKYB101ELL102MM40S; footprint Custom:C320C105K5R5TA -> Custom:EKYB101ELL102MM40S
- C38: value EKYB101ELL102MM40S -> 4.7uF; footprint Custom:EKYB101ELL102MM40S -> Capacitor_THT:C_Rect_L7.0mm_W2.5mm_P5.00mm
- C40: value EKYB101ELL102MM40S -> 10nF; footprint Custom:EKYB101ELL102MM40S -> Capacitor_THT:C_Rect_L4.0mm_W2.5mm_P2.50mm
- C41: value EKYB101ELL102MM40S -> 1000uF; footprint Custom:EKYB101ELL102MM40S -> Custom:ECA-1JM102
- C42, C44: value EKYB101ELL102MM40S -> 0.1uF; footprint Custom:EKYB101ELL102MM40S -> Capacitor_THT:C_Rect_L7.0mm_W2.5mm_P5.00mm
- C43: value EKYB101ELL102MM40S -> 470uF; footprint Custom:EKYB101ELL102MM40S -> Custom:UPW1E471MPD6TA
- C45, C46: value ~ -> 0.1uF
- C47: value R75RR322050L4J -> 10uF; footprint Custom:R75RR322050L4J -> Capacitor_THT:C_Rect_L4.0mm_W2.5mm_P2.50mm
- C48: value R75RR322050L4J -> 4.7nF; footprint Custom:R75RR322050L4J -> Capacitor_THT:C_Rect_L7.0mm_W2.5mm_P5.00mm
- C49: value R75RR322050L4J -> 1000uF; footprint Custom:R75RR322050L4J -> Custom:ECA-1JM102
- C50, C52: value R75RR322050L4J -> 0.1uF; footprint Custom:R75RR322050L4J -> Capacitor_THT:C_Rect_L7.0mm_W2.5mm_P5.00mm
- C51: value R75RR322050L4J -> 470uF; footprint Custom:R75RR322050L4J -> Custom:UPW1E471MPD6TA
- D1: value MBR40250G -> 1N4148; footprint Custom:MBR40250G -> Diode_THT:D_DO-35_SOD27_P10.16mm_Horizontal
- D2, D3: value ~ -> 1N4148; footprint Diode_THT:D_DO-35_SOD27_P7.62mm_Horizontal -> Diode_THT:D_DO-35_SOD27_P10.16mm_Horizontal
- D4: value 1N4148 -> BZX55C3V0-TR; footprint Diode_THT:D_DO-35_SOD27_P7.62mm_Horizontal -> Diode_THT:D_DO-35_SOD27_P10.16mm_Horizontal
- D5: value 1N4148 -> 1N5822; footprint Diode_THT:D_DO-35_SOD27_P7.62mm_Horizontal -> Diode_THT:D_DO-201AD_P12.70mm_Horizontal
- D6: value 1N4148 -> 1N4149; footprint Diode_THT:D_DO-35_SOD27_P7.62mm_Horizontal -> Diode_THT:D_DO-35_SOD27_P10.16mm_Horizontal
- D8: value MBR40250G -> 1N4149; footprint Custom:MBR40250G -> Diode_THT:D_DO-35_SOD27_P10.16mm_Horizontal
- H1: value Heatsink 1 -> Heatsink
- H2: value Heatsink 2 -> Heatsink
- J1: value SCL, SDA, +, GND -> Vsupply; footprint Connector_PinHeader_2.54mm:PinHeader_1x04_P2.54mm_Vertical -> Custom:PCB-3 (M4)
- J10: value USB RWGBS -> Tap debug pin; footprint Custom:USB connection -> Connector_PinHeader_2.54mm:PinHeader_1x01_P2.54mm_Vertical
- J14: value Standoff Hole -> Conn_01x01_Pin; footprint Custom:ContactViaM3 -> Custom:PCB-3 (M4)
- J15: value Standoff Hole -> Tap; footprint Custom:ContactViaM3 -> Custom:PCB-1 (M4)
- J2: value Conn_01x08_Pin -> GND; footprint Connector_PinHeader_2.54mm:PinHeader_1x08_P2.54mm_Vertical -> Custom:PCB-3 (M4)
- J3: value Conn_01x01_Pin -> ~; footprint Custom:5055556-9 -> Connector_PinHeader_2.54mm:PinHeader_1x01_P2.54mm_Vertical
- J4: value Conn_01x01_Pin -> Conn_01x08_Pin; footprint Custom:5055556-9 -> Connector_PinHeader_2.54mm:PinHeader_1x08_P2.54mm_Vertical
- J5: value +36V -> ~; footprint Custom:5055556-9 -> Connector_PinHeader_2.54mm:PinHeader_1x01_P2.54mm_Vertical
- J6: value GND -> ~; footprint Custom:5055556-9 -> Connector_PinHeader_2.54mm:PinHeader_1x01_P2.54mm_Vertical
- J8: value Conn_01x04_Pin -> SCL, SDA, +, GND; footprint TerminalBlock:TerminalBlock_MaiXu_MX126-5.0-04P_1x04_P5.00mm -> Connector_PinHeader_2.54mm:PinHeader_1x04_P2.54mm_Vertical
- J9: value USB RWGBS -> Tap; footprint Custom:USB connection -> Custom:PCB-1 (M4)
- L2: value 74436411500 -> 68uH; footprint Custom:74436411500 -> Custom:5026 Inductor
- R1: value R_drive 5 -> ~; footprint Resistor_THT:R_Axial_DIN0207_L6.3mm_D2.5mm_P10.16mm_Horizontal -> Custom:RX24-100W
- R10: value R_pcfb_in 1K -> Pullup
- R11: value R_pcfb_f 56K -> 1K
- R12: value R_pfb_i 1K -> 2K 1%
- R13: value R_sfb_i 1K -> 120K
- R14: value R_pulldown 1000 -> 1K
- R15: value 3K -> 2K 1%
- R16: value 1K -> 10; footprint Resistor_THT:R_Axial_DIN0207_L6.3mm_D2.5mm_P7.62mm_Horizontal -> Custom:SL2TTED10R0F
- R17: value 1.33K -> 50; footprint Resistor_THT:R_Axial_DIN0309_L9.0mm_D3.2mm_P12.70mm_Horizontal -> Resistor_THT:R_Axial_DIN0207_L6.3mm_D2.5mm_P7.62mm_Horizontal
- R18: value Pullup -> 100
- R19: value Pullup -> 1K
- R2: value R_sfb_H 500K -> 1.33K
- R3: value R_sfb_L 6.8K -> 33k
- R4: value ~ -> 1K; footprint Custom:RX24-100W -> Resistor_THT:R_Axial_DIN0207_L6.3mm_D2.5mm_P7.62mm_Horizontal
- R5: value 1.33K -> 1K; footprint Resistor_THT:R_Axial_DIN0309_L9.0mm_D3.2mm_P12.70mm_Horizontal -> Resistor_THT:R_Axial_DIN0207_L6.3mm_D2.5mm_P7.62mm_Horizontal
- R6: value 10K -> 2k
- R7: value R_pfb_H 270K -> 1.33K
- R8: value R_pfb_ 10K -> 10K
- R9: value R_pcfb_sense 0.001 -> Pullup; footprint Custom:PCS2512FR0010ET -> Resistor_THT:R_Axial_DIN0207_L6.3mm_D2.5mm_P7.62mm_Horizontal
- U1: footprint Package_DIP:CERDIP-8_W7.62mm_SideBrazed_LongPads -> Package_TO_SOT_THT:TO-92
- U2: footprint Package_DIP:CERDIP-8_W7.62mm_SideBrazed_LongPads -> Custom:ESP32_WROOM-32_Dev_Board
- U3: footprint Package_TO_SOT_THT:TO-92 -> Package_TO_SOT_THT:TO-220-5_Vertical
- U4: footprint Custom:IXFP60N25X3 -> Package_TO_SOT_THT:TO-92
- U5: footprint Package_TO_SOT_THT:TO-92 -> Package_DIP:DIP-20_W7.62mm_Socket_LongPads
- U6: footprint Custom:AWHSH124D00G -> Package_TO_SOT_THT:TO-220-5_Vertical
- U7: footprint Custom:AWHSH124D00G -> Package_TO_SOT_THT:TO-92
- moved J4 482.3 mm to (543.9, 152.6)
- moved C49 430.1 mm to (476.2, 149.2)
- moved C50 385.1 mm to (465.8, 155.5), turned to 90 degrees
- moved J3 363.5 mm to (439.8, 121.2)
- moved C51 362.7 mm to (444.8, 146.0), turned to 90 degrees
- moved U3 361.9 mm to (465.0, 132.0), turned to 180 degrees
- moved R15 361.2 mm to (447.8, 163.0), turned to 90 degrees
- moved C52 359.9 mm to (442.8, 152.5)
- moved U4 350.5 mm to (389.3, -10.4)
- moved J8 330.2 mm to (359.0, 7.52), turned to 0 degrees
- moved L2 319.5 mm to (450.8, 121.2), turned to 0 degrees
- moved C41 312.8 mm to (476.2, 120.5), turned to 0 degrees
- moved R12 300.5 mm to (447.8, 134.3), turned to 90 degrees
- moved C48 284.2 mm to (94.2, -108.4)
- moved D5 283.7 mm to (461.2, 126.8), turned to 90 degrees
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- renumbered J11 to J20, J12 to J22, J13 to J23
Connections:
- C1 pad 1: Earth -> +36V
- C1 pad 2: +10V -> Earth
- C10 pad 1: Net-(OR3-Vout) -> +36V
- C11 pad 1: +3V3 -> Net-(OR1-Vout)
- C12 pad 1: Net-(OR4-Vout) -> Net-(OR2-Vout)
- C13 pad 1: +3V3 -> Net-(OR3-Vout)
- C14 pad 1: +3V3 -> Net-(OR4-Vout)
- C16 pad 1: +3V3 -> Net-(OR6-Vout)
- C17 pad 1: Net-(OR6-Vout) -> +3V3
- C2 pad 1: +3V3 -> +36V
- C20 pad 1: Net-(D1-K) -> +3V3
- C21 pad 1: Net-(D1-K) -> +3V3
- C22 pad 1: Net-(D1-K) -> +3V3
- C23 pad 1: Net-(D1-K) -> +3V3
- C24 pad 1: Net-(U3-Cathode) -> +3V3
- C28 pad 1: +3V3 -> +36V
- C29 pad 1: Net-(D1-K) -> +36V
- C3 pad 1: +10V -> +36V
- C30 pad 1: Net-(D1-K) -> +36V
- C31 pad 1: Net-(D1-K) -> +36V
- C32 pad 1: Net-(D1-K) -> +36V
- C33 pad 1: Net-(D1-K) -> +36V
- C34 pad 1: Net-(D1-K) -> +36V
- C35 pad 1: Net-(D1-K) -> +36V
- C36 pad 1: Net-(D1-K) -> +36V
- C37 pad 1: Net-(D1-K) -> +36V
- C38 pad 1: Net-(D1-K) -> Net-(D4-K)
- C4 pad 1: +3V3 -> +36V
- C40 pad 1: Net-(D1-K) -> Net-(U3-FEEDBACK)
- C40 pad 2: Earth -> +3V3
- C41 pad 1: Net-(D1-K) -> Net-(U3-VIN)
- C42 pad 1: Net-(D1-K) -> Net-(U3-VIN)
- C43 pad 1: Net-(D1-K) -> +3V3
- C44 pad 1: Net-(D1-K) -> +3V3
- C45 pad 1: Net-(OR7-Vout) -> Net-(U4-Cathode)
- C47 pad 1: Net-(D1-A) -> +3V3
- C47 pad 2: Net-(J4-Pin_1) -> Earth
- C48 pad 1: Net-(D1-A) -> Net-(U6-FEEDBACK)
- C48 pad 2: Net-(J4-Pin_1) -> +5V
- C49 pad 1: Net-(D1-A) -> Net-(U6-VIN)
- C49 pad 2: Net-(J4-Pin_1) -> Earth
- C5 pad 1: +3V3 -> +36V
- C50 pad 1: Net-(D1-A) -> Net-(U6-VIN)
- C50 pad 2: Net-(J4-Pin_1) -> Earth
- C51 pad 1: Net-(D1-A) -> +5V
- C51 pad 2: Net-(J4-Pin_1) -> Earth
- C52 pad 1: Net-(D1-A) -> +5V
- C52 pad 2: Net-(J4-Pin_1) -> Earth
- C6 pad 1: Net-(OR1-Vout) -> +36V
- C7 pad 1: Net-(OR2-Vout) -> +36V
- C8 pad 1: +3V3 -> +36V
- C9 pad 1: +3V3 -> +36V
- D2 pad 1: Net-(D2-Pad1) -> Net-(D2-K)
- D3 pad 1: Net-(D3-Pad1) -> Net-(D3-K)
- D3 pad 2: Earth -> Net-(D3-A)
- D4 pad 2: Net-(D4-A) -> Earth
- D6 pad 1: Net-(D6-K) -> Net-(D12-K)
- D8 pad 1: Net-(D8-K) -> Net-(D7-K)
- D8 pad 2: Earth -> Net-(D11-K)
- F1 pad 1: Net-(J5-Pin_1) -> Net-(J1-Pin_1)
- F1 pad 2: Net-(D6-A) -> Net-(D1-A)
- H1 pad 1: Earth -> +36V
- H2 pad 1: Net-(D1-K) -> +36V
- J1 pad 1: Earth -> Net-(J1-Pin_1)
- J10 pad 1: Net-(J10-Pin_1) -> Net-(D6-A)
- J14 pad 1: Earth -> Net-(J14-Pin_1)
- J15 pad 1: Earth -> Net-(D12-A)
- J2 pad 1: +3V3 -> Earth
- J3 pad 1: Net-(D1-K) -> +3V3
- J4 pad 1: Net-(J4-Pin_1) -> +3V3
- J5 pad 1: Net-(J5-Pin_1) -> +5V
- J6 pad 1: Earth -> +15V
- J8 pad 2: Earth -> +3V3
- J8 pad 3: Net-(D4-K) -> Net-(J4-Pin_4)
- J8 pad 4: +10V -> Net-(J4-Pin_3)
- J9 pad 1: Net-(J9-Pin_1) -> Net-(D6-A)
- L1 pad 1: Net-(L1-Pad1) -> Net-(K2-Pad4)
- L1 pad 2: Net-(D1-K) -> +36V
- L2 pad 1: Net-(D8-K) -> +3V3
- L2 pad 2: Net-(D1-A) -> Net-(D5-K)
- R1 pad 1: Net-(R1-Pad1) -> Net-(D3-K)
- R1 pad 2: Net-(U4-G) -> Net-(K2-Pad4)
- R10 pad 1: Net-(U2-VIN-) -> +3V3
- R10 pad 2: Earth -> Net-(J4-Pin_4)
- R11 pad 1: Net-(U2-VOUT) -> +3V3
- R11 pad 2: Net-(U2-VIN-) -> Net-(U4-Cathode)
- R12 pad 1: Net-(X1-D35_a1i) -> Net-(U3-FEEDBACK)
- R12 pad 2: Net-(D3-Pad1) -> Earth
- R13 pad 1: Net-(X1-VP_a1i) -> Net-(D6-A)
- R13 pad 2: Net-(D2-Pad1) -> Net-(R13-Pad2)
- R14 pad 1: Net-(R1-Pad1) -> +3V3
- R14 pad 2: Earth -> Net-(U12-VREF_IN/OUT)
- R15 pad 1: +3V3 -> Net-(U6-FEEDBACK)
- R15 pad 2: Net-(U3-Cathode) -> Earth
- R16 pad 1: Net-(X1-D13_a2io) -> Net-(D7-K)
- R16 pad 2: Net-(U5-G) -> Earth
- R17 pad 1: Net-(D6-K) -> +3V3
- R17 pad 2: Net-(D5-K) -> Net-(D12-K)
- R18 pad 1: +3V3 -> Net-(D12-K)
- R18 pad 2: Net-(J1-Pin_3) -> Earth
- R19 pad 2: Net-(J1-Pin_4) -> Net-(U18-Cathode)
- R2 pad 1: Net-(J4-Pin_1) -> Net-(D1-K)
- R2 pad 2: Net-(D2-Pad1) -> Net-(D2-K)
- R3 pad 1: Net-(D2-Pad1) -> +36V
- R3 pad 2: Earth -> Net-(D4-K)
- R4 pad 1: Net-(D4-K) -> Net-(U2-D35_a1i)
- R4 pad 2: Net-(L1-Pad1) -> Net-(D4-K)
- R5 pad 1: Net-(D4-A) -> Net-(U2-D21_io)
- R5 pad 2: Net-(U5-D) -> Net-(U1-G)
- R6 pad 1: Net-(X1-D13_a2io) -> Net-(D4-K)
- R7 pad 1: Net-(D1-K) -> Net-(D3-A)
- R7 pad 2: Net-(D3-Pad1) -> Net-(U1-D)
- R8 pad 1: Net-(D3-Pad1) -> Net-(U2-D21_io)
- R9 pad 1: Net-(U2-VIN+) -> +3V3
- R9 pad 2: Earth -> Net-(J4-Pin_3)
- S1 pad 1: Net-(J9-Pin_1) -> Net-(J7-VCC)
- S1 pad 2: Net-(J10-Pin_1) -> Net-(J3-VCC)
- S1 pad 5: +3V3 -> +5V
- U1 pad 1: +10V -> Earth
- U1 pad 2: Net-(U1-IN) -> Net-(U1-G)
- U1 pad 3: unconnected-(U1-NC-Pad3) -> Net-(U1-D)
- U2 pad 2: Net-(U2-VIN-) -> Net-(OR2-Vout)
- U2 pad 3: Net-(U2-VIN+) -> Net-(OR1-Vout)
- U2 pad 4: Earth -> Net-(U17-69)
- U2 pad 5: unconnected-(U2-NC-Pad5) -> Net-(U2-D35_a1i)
- U2 pad 6: Net-(U2-VOUT) -> Net-(U11-DIN)
- U2 pad 7: +3V3 -> Net-(U2-D33_a1io)
- U2 pad 8: unconnected-(U2-NC-Pad8) -> Net-(U17-60)
- U3 pad 1: unconnected-(U3-NC-Pad1) -> Net-(U3-VIN)
- U3 pad 2: Net-(U3-Cathode) -> Net-(D5-K)
- U4 pad 1: Net-(U4-G) -> unconnected-(U4-NC-Pad1)
- U4 pad 2: Net-(J4-Pin_1) -> Net-(U4-Cathode)
- U4 pad 3: Net-(U2-VIN+) -> Earth
- U5 pad 1: Earth -> Net-(U17-84)
- U5 pad 2: Net-(U5-G) -> Net-(U17-74)
- U5 pad 3: Net-(U5-D) -> Net-(U17-72)
- U6 pad 1: Net-(D4-A) -> Net-(U6-VIN)
- U6 pad 2: Net-(D4-K) -> Net-(D10-K)
- U6 pad 3: Net-(D4-K) -> Earth
- U6 pad 4: Net-(L1-Pad1) -> Net-(U6-FEEDBACK)
- U6 pad 5: unconnected-(U6-Pad5) -> Earth
- U7 pad 1: Earth -> unconnected-(U7-NC-Pad1)
- U7 pad 2: Net-(D6-A) -> Net-(U12-VREF_IN/OUT)
- U7 pad 3: Net-(D5-K) -> Earth
Routing:
- net +3V3: track 539.6 -> 21.8 mm, vias 3 -> 0
- net Net-(D1-K): track 296.0 -> 0.00 mm, vias 123 -> 0
- net Net-(D4-K): track 268.3 -> 0.00 mm, vias 11 -> 0
- net Net-(OR7-Vout): track 138.5 -> 0.00 mm
- net Net-(OT4-Vin): track 134.5 -> 0.00 mm
- net Net-(OR6-Vout): track 116.0 -> 0.00 mm
- net Net-(OR5-Vout): track 104.1 -> 0.00 mm
- net Net-(OT3-Vin): track 100.0 -> 0.00 mm
- net Net-(J5-Pin_1): track 96.6 -> 0.00 mm, vias 11 -> 0
- net Net-(H3-Pin_1): track 0.00 -> 93.2 mm
- net Net-(D7-K): track 0.00 -> 84.8 mm, vias 0 -> 2
- net Net-(U17-28): track 0.00 -> 83.6 mm
- net +5V: track 0.00 -> 83.0 mm
- net Net-(OR4-Vout): track 81.4 -> 0.00 mm
- net Net-(U17-135): track 0.00 -> 78.8 mm
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- removed copper zone on F.Cu, net Earth
- removed copper zone on B.Cu, net Net-(D1-A)
- removed copper zone on F.Cu, net Net-(D1-A)
- removed copper zone on B.Cu, net Net-(D1-K)
- removed copper zone on F.Cu, net Net-(D1-K)
- removed copper zone on B.Cu, net Net-(D8-K)
- removed copper zone on F.Cu, net Net-(D8-K)
- removed copper zone on B.Cu, net Net-(J4-Pin_1)
- removed copper zone on F.Cu, net Net-(J4-Pin_1)
- removed copper zone on B.Cu, net Net-(J5-Pin_1)
- removed copper zone on B.Cu, net Net-(L1-Pad1)
- removed copper zone on F.Cu, net Net-(L1-Pad1)
- removed copper zone on B.Cu, net Net-(U2-VIN+)
- removed copper zone on F.Cu, net Net-(U2-VIN+)
Other:
- board size 234.5 x 198.2 mm -> 302.3 x 198.2 mm
- board text added: "Floating On Live"
- board text added: "Floating On Tap"
- board text removed: "Ext USB S B G W R"
- board text removed: "FB+"
- board text removed: "FB-"
- board text removed: "First Stage Voltage Feedback"
- board text removed: "GND GND Vin 10V"
- board text removed: "GND GND Vin 3.3V"
- board text removed: "HEAT SINK LIVE"
- board text removed: "HJP+GPT"
- board text removed: "I2C SCL,SDA,GND,3.3V"
- board text removed: "In+"
- board text removed: "In- GND"
- board text removed: "Insulating layer must be added here under power resistor."
- board text removed: "Int USB"
- board text removed: "One Stone Solutions LTD"
- board text removed: "Other Peripherals"
- board text removed: "Output Current Feedback"
- board text removed: "Output Voltage Feedback"
- board text removed: "PS pwr"
- board text removed: "USB pwr"

Commit message: PCB coming together :)
Parts:
- added C39: 1000uF, Custom:ECA-1JM102, F.Cu at (488.6, 205.5)
- added C77: 0.1uF, Capacitor_THT:C_Rect_L7.0mm_W2.5mm_P5.00mm, F.Cu at (481.4, 223.3)
- added C78: 470uF, Custom:UPW1E471MPD6TA, F.Cu at (484.6, 255.0)
- added C79: 2.2nF, Capacitor_THT:C_Rect_L7.0mm_W2.5mm_P5.00mm, F.Cu at (481.4, 227.4)
- added C80: 0.1uF, Capacitor_THT:C_Rect_L7.0mm_W2.5mm_P5.00mm, F.Cu at (481.4, 231.4)
- added C81: 0.1uF, Capacitor_THT:C_Rect_L7.0mm_W2.5mm_P5.00mm, F.Cu at (117.2, 219.0)
- added C82: 0.1uF, Capacitor_THT:C_Rect_L7.0mm_W2.5mm_P5.00mm, F.Cu at (141.5, 219.0)
- added D17: 1N5822, Diode_THT:D_DO-201AD_P12.70mm_Horizontal, F.Cu at (481.9, 217.9)
- added J7: ~, Connector_PinHeader_2.54mm:PinHeader_1x01_P2.54mm_Vertical, F.Cu at (492.0, 252.2)
- added L8: ~, Custom:5026 Inductor, F.Cu at (481.4, 188.4)
- added L9: 68uH, Custom:5026 Inductor, F.Cu at (491.0, 188.4)
- added R38: 2K 1%, Resistor_THT:R_Axial_DIN0207_L6.3mm_D2.5mm_P7.62mm_Horizontal, F.Cu at (481.1, 247.9)
- added RV6: 30K, Potentiometer_THT:Potentiometer_Bourns_3296W_Vertical, F.Cu at (487.7, 242.7)
- added U28: ~, Custom:HW-677 LM2596HVS DC-DC, F.Cu at (125.9, 95.0)
- added U29: ~, Custom:HW-677 LM2596HVS DC-DC, F.Cu at (184.7, 95.0)
- added U30: ~, Custom:HW-677 LM2596HVS DC-DC, F.Cu at (235.3, 95.0)
- added U31: ~, Custom:HW-677 LM2596HVS DC-DC, F.Cu at (237.9, 233.8)
- added U32: ~, Package_TO_SOT_THT:TO-220-5_Vertical, F.Cu at (481.9, 237.4)
- R21, R22, R30, R31: value 6.2 -> 4.7
- moved U4 352.6 mm to (121.0, 218.4)
- moved J3 334.9 mm to (106.2, 91.9)
- moved C42 333.9 mm to (133.2, 97.4)
- moved D5 333.9 mm to (128.7, 97.5)
- moved U3 333.9 mm to (132.4, 102.7)
- moved C43 333.9 mm to (112.2, 87.9)
- moved C44 333.9 mm to (110.2, 94.4)
- moved L2 333.9 mm to (118.2, 91.9)
- moved R12 333.9 mm to (115.2, 105.0)
- moved RV1 333.9 mm to (110.2, 99.2)
- moved C41 333.1 mm to (143.9, 97.2)
- moved R13 332.7 mm to (117.3, 224.2), turned to 180 degrees
- moved U18 330.8 mm to (145.0, 218.4)
- moved R27 329.1 mm to (141.6, 224.2), turned to 180 degrees
- moved C47 316.4 mm to (124.2, 207.2), turned to 90 degrees
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Connections:
- R37 pad 1: +15V -> +14V
- U23 pad 10: Net-(U17-135) -> Net-(U17-143)
- U23 pad 11: Net-(U17-143) -> Net-(U17-141)
- U23 pad 12: Net-(U17-141) -> Net-(U17-135)
- U24 pad 10: Net-(U17-141) -> Net-(U17-135)
- U24 pad 11: Net-(U17-143) -> Net-(U17-141)
- U24 pad 12: Net-(U17-135) -> Net-(U17-143)
Routing:
- net Net-(U17-141): track 24.8 -> 203.3 mm, vias 0 -> 1
- net +3V3: track 21.8 -> 184.1 mm
- net Net-(U17-143): track 68.4 -> 202.3 mm
- net +36V: track 73.1 -> 202.9 mm
- net Net-(U17-135): track 78.8 -> 199.9 mm, vias 0 -> 1
- net unconnected-(U24-Pad4): track 71.2 -> 0.00 mm
- net Net-(D6-A): track 0.00 -> 32.7 mm
- net Net-(D12-A): track 0.00 -> 31.6 mm
- net unconnected-(U17-137!-Pad64): track 30.5 -> 0.00 mm
- net Net-(U19-VIN): track 14.1 -> 38.7 mm
- net Net-(U28-IN+): track 15.0 -> 39.4 mm
- net Net-(U29-IN+): track 15.1 -> 37.1 mm
- net Earth: track 123.3 -> 141.0 mm, vias 49 -> 53
- net Net-(H3-Pin_1): track 93.2 -> 110.7 mm
- net +15V: track 42.0 -> 54.5 mm, vias 0 -> 1
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Other:
- board text added: "3.3V"
- board text added: "5V"

Commit message: Going great.
Parts:
- removed S1: ~, Custom:SLW-1678105-6A-N-D
- C54, R14: moved to B.Cu
- D1, D2, D3: footprint Diode_THT:D_DO-35_SOD27_P10.16mm_Horizontal -> Diode_THT:D_DO-35_SOD27_P7.62mm_Horizontal
- D12, D6: footprint Diode_THT:D_DO-35_SOD27_P10.16mm_Horizontal -> Diode_THT:D_DO-35_SOD27_P5.08mm_Vertical_AnodeUp
- moved J4 478.8 mm to (67.8, 102.0), turned to 90 degrees
- moved R3 352.9 mm to (77.8, 247.7), turned to 180 degrees
- moved R4 350.5 mm to (46.8, 245.7), turned to -90 degrees
- moved C38 331.4 mm to (72.6, 237.0)
- moved D4 324.2 mm to (67.6, 240.3)
- moved C39 309.3 mm to (180.4, 232.0), turned to 180 degrees
- moved J8 309.2 mm to (67.8, 111.4)
- moved C66 307.3 mm to (152.8, 206.9), turned to 90 degrees
- moved J7 294.5 mm to (207.7, 329.2)
- moved C40 294.0 mm to (88.5, 203.0)
- moved C77 290.3 mm to (191.2, 231.8), turned to -90 degrees
- moved U32 290.2 mm to (191.9, 226.6)
- moved L9 289.0 mm to (206.2, 237.3), turned to 180 degrees
- moved D17 286.6 mm to (195.7, 231.8), turned to -90 degrees
- moved R14 285.1 mm to (180.4, 172.7), turned to 180 degrees
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Connections:
- C74 pad 2: +15V -> +14V
- R29 pad 1: Net-(U2-D33_a1io) -> Net-(U25-G)
- R8 pad 1: Net-(U2-D21_io) -> Net-(U1-G)
- S2 pad 1: Net-(J12-Pin_1) -> Net-(J11-Pin_1)
- S2 pad 2: Net-(J11-Pin_1) -> Net-(J12-Pin_1)
- U12 pad 5: Net-(U12-!CS) -> Earth
- U17 pad 12: Net-(U17-38) -> Net-(OT5-Vin)
- U17 pad 56: Net-(OT4-Vin) -> Net-(U17-3)
- U17 pad 58: Net-(OT5-Vin) -> Net-(U12-DB3)
- U17 pad 6: Net-(U17-28) -> Net-(OT4-Vin)
- U17 pad 60: Net-(U17-143) -> Net-(U12-DB4)
- U17 pad 62: Net-(U17-141) -> Net-(U12-DB5)
- U17 pad 66: Net-(U17-135) -> Net-(U12-DB6)
- U17 pad 72: Net-(U12-DB6) -> Net-(U12-DB2)
- U17 pad 73: Net-(U12-!EOC) -> Net-(U17-125)
- U17 pad 74: Net-(U12-DB5) -> Net-(U12-DB1)
- U17 pad 75: Net-(U12-!RD) -> Net-(U17-121)
- U17 pad 76: Net-(U12-DB4) -> Net-(U12-DB0)
- U17 pad 80: Net-(U12-DB3) -> Net-(U12-!CONVST)
- U17 pad 81: Net-(U12-!CS) -> Net-(U17-112)
- U17 pad 82: Net-(U12-DB0) -> Net-(U12-!RD)
- U17 pad 83: Net-(U12-!CONVST) -> Net-(U17-110)
- U17 pad 84: Net-(U12-DB1) -> Net-(U12-!EOC)
- U17 pad 86: Net-(U12-DB2) -> Net-(U17-104)
- U20 pad 16: Net-(U17-127) -> Net-(U17-121)
- U20 pad 17: Net-(U17-129) -> Net-(U17-125)
- U20 pad 18: Net-(U17-142) -> Net-(U17-127)
- U20 pad 19: Net-(U17-144) -> Net-(U17-129)
- U20 pad 2: Net-(U17-38) -> Net-(U17-44)
- U20 pad 20: Net-(U17-2) -> Net-(U17-142)
- U20 pad 3: Net-(U17-28) -> Net-(U17-49)
- U20 pad 4: Net-(U17-44) -> Net-(U17-51)
- U20 pad 5: Net-(U17-49) -> Earth
- U20 pad 6: Net-(U17-51) -> Net-(U17-53)
- U20 pad 8: Net-(U17-53) -> Net-(U17-55)
- U23 pad 10: Net-(U17-143) -> Net-(U17-144)
- U23 pad 11: Net-(U17-141) -> Net-(U17-2)
- U23 pad 12: Net-(U17-135) -> Net-(U17-3)
- U24 pad 10: Net-(U17-135) -> Net-(U17-112)
- U24 pad 11: Net-(U17-141) -> Net-(U17-110)
- U24 pad 12: Net-(U17-143) -> Net-(U17-104)
- U24 pad 3: +15V -> +14V
- U5 pad 1: Net-(U17-84) -> Net-(U17-85)
- U5 pad 16: Net-(U17-55) -> Net-(U17-59)
- U5 pad 17: Net-(U17-59) -> Net-(U17-64)
- U5 pad 18: Net-(U17-64) -> Net-(U17-68)
- U5 pad 19: Net-(U17-68) -> Net-(U17-70)
- U5 pad 2: Net-(U17-74) -> Net-(U17-84)
- U5 pad 20: Net-(U17-70) -> Net-(U17-72)
- U5 pad 3: Net-(U17-72) -> Net-(U17-74)
- U5 pad 4: Net-(U17-85) -> Net-(U17-83)
- U5 pad 5: Net-(U17-83) -> Earth
Routing:
- net +3V3: track 184.1 -> 469.1 mm, vias 0 -> 1
- net Net-(U17-141): track 203.3 -> 0.00 mm, vias 1 -> 0
- net Net-(U17-143): track 202.3 -> 0.00 mm
- net Net-(U17-135): track 199.9 -> 0.00 mm, vias 1 -> 0
- net +5V: track 84.0 -> 207.7 mm
- net Net-(U17-112): track 0.00 -> 113.2 mm, vias 0 -> 2
- net Net-(U17-110): track 0.00 -> 105.1 mm, vias 0 -> 2
- net Net-(U17-104): track 0.00 -> 95.8 mm, vias 0 -> 2
- net Net-(U17-28): track 83.6 -> 0.00 mm
- net Net-(OR4-Vout): track 5.10 -> 88.1 mm
- net Net-(U17-38): track 71.9 -> 0.00 mm
- net Net-(U17-55): track 0.00 -> 71.7 mm
- net Net-(U17-53): track 0.00 -> 69.9 mm
- net Net-(U17-3): track 0.00 -> 67.8 mm
- net Net-(OR5-Vout): track 6.49 -> 71.1 mm
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- added copper zone on F.Cu, net +36V
- added copper zone on F.Cu, net Earth
Other:
- board size 302.3 x 198.2 mm -> 305.3 x 178.2 mm
