File: Kicad/HVPSController2/HVPSController2.kicad_sch (KiCad schematic)
At the start: 117 parts, among them J1 SCL, SDA, +, GND, J10 USB RWGBS, J11 Standoff Hole, J12 Standoff Hole, J13 Standoff Hole, J14 Standoff Hole, J15 Standoff Hole, J2 Conn_01x08_Pin, J3 Conn_01x01_Pin, J4 Conn_01x01_Pin, J5 Vsupply, J6 GND, J7 Conn_01x04_Pin, J8 Conn_01x04_Pin, J9 USB RWGBS

Commit message: Voltage regulators designed!
Parts:
- removed U2: ~, Package_DIP:CERDIP-8_W7.62mm_SideBrazed_LongPads, symbol Custom:MCP6021-E/P
- added C26, C48, C50, C53, C56, C58: 470uF, symbol Device:C_Polarized
- added C47, C49, C52, C55, C57, C60: 0.1uF, Custom:C320C105K5R5TA, symbol Device:C
- added C51: 10nF, Custom:C320C105K5R5TA, symbol Device:C
- added C54: 4.7nF, Custom:C320C105K5R5TA, symbol Device:C
- added C59: 2.2nF, Custom:C320C105K5R5TA, symbol Device:C
- added D1, D2, D7, D8: 1N4149, Diode_THT:D_DO-35_SOD27_P7.62mm_Horizontal, symbol Diode:1N4149
- added D10, D11, D9: 1N5822, Diode_THT:D_DO-201AD_P15.24mm_Horizontal, symbol Diode:1N5822
- added L2, L3, L4: 68uH, symbol Device:L
- added R23: 2K 1%, symbol Device:R
- added RV1: 5K, symbol Device:R_Potentiometer
- added RV2: 10K, symbol Device:R_Potentiometer
- added RV3: 20K, symbol Device:R_Potentiometer
- added U13: ~, symbol Custom:CST2020-200L
- added U14, U15, U16: ~, symbol Custom:LM2596HV
- added U2: ~, symbol Custom:AD7822
- R10: value R_pcfb_in 1K -> 2K 1%; footprint Resistor_THT:R_Axial_DIN0207_L6.3mm_D2.5mm_P7.62mm_Horizontal -> (none)
- R11: value R_pcfb_f 56K -> 2K 1%; footprint Resistor_THT:R_Axial_DIN0207_L6.3mm_D2.5mm_P7.62mm_Horizontal -> (none)
- R9: value R_pcfb_sense 0.001 -> 10; footprint Custom:PCS2512FR0010ET -> (none)
Connections:
- net +36V: now also C26.1, C47.1, C50.1, C52.1, C56.1, C57.1, U14.1 (VIN), U15.1 (VIN), U16.1 (VIN)
- net +3V3: now also U2.14 (VDD)
- net Earth: now also R11.2, C26.2, C47.2, C48.2, C49.2, C50.2, C52.2, C53.2, C55.2, C56.2, C57.2, C58.2, C60.2, D10.2 (A), D11.2 (A), D7.2 (A), D8.2 (A), D9.2 (A), R23.2, U14.3 (GND), U14.5 (ON/OFF), U15.3 (GND), U15.5 (ON/OFF), U16.3 (GND), U16.5 (ON/OFF), U2.15 (AGND), U2.7 (DGND)
- net at R20.2, U4.2 (D), U8.3 (S): now also U13.5; no longer J3.1 (Pin_1)
- net at R9.1: now also D1.1 (K), D2.1 (K), U2.11 (VIN1)
- net at R10.1: now also C51.1, RV1.2, U14.4 (FEEDBACK); no longer R11.2
- net at R11.1: now also C54.1, RV2.2, U15.4 (FEEDBACK); no longer X1.4 (D34_a1i)
- new net: D11.1 (K), L4.2, U16.2 (OUTPUT)
- new net: C58.1, C59.2, C60.1, L4.1, RV3.1
- new net: C48.1, C49.1, C51.2, L2.1, RV1.1
- new net: D10.1 (K), L3.2, U15.2 (OUTPUT)
- new net: C59.1, R23.1, RV3.2, U16.4 (FEEDBACK)
- new net: C53.1, C54.2, C55.1, L3.1, RV2.1
- new net: D9.1 (K), L2.2, U14.2 (OUTPUT)
- new net: D2.2 (A), D8.1 (K), U13.1
- new net: D1.2 (A), D7.1 (K), U13.3
Other:
- note added: "10V Regulator"
- note added: "3.3V Regulator"
- note added: "5V Regulator"
- moved on the sheet: C1, C19, C25, C28, H1, H2, H3, H5, J11, J12, J13, J14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

Commit message: Verified safe fpga pins for io all on 3.3v bus. Maths for H-Bridge going nicely :)
I let gpt produce a list from reading the data sheet and then manually verified all pins im using are safe.
Parts:
- removed C45: ~, Capacitor_THT:C_Rect_L7.0mm_W2.5mm_P5.00mm, symbol Custom:C317C300J5G5TA
- removed OR7: ~, Custom:RS PRO Optical Receiver jack, symbol Custom:RS_PRO_Optical_Receiver_jack
- added C45: ~, Capacitor_THT:C_Rect_L7.0mm_W2.5mm_P5.00mm, symbol Custom:C322C104J5R5TA
- added C61: 0.1uF, Capacitor_THT:C_Disc_D7.0mm_W2.5mm_P5.00mm, symbol Device:C
- added C62, C63: 10uF, Custom:C320C105K5R5TA, symbol Device:C
- added C64, C65, C66, C67: ~, Custom:C320C105K5R5TA, symbol Device:C
- added D12, D13: 1N4149, Diode_THT:D_DO-35_SOD27_P7.62mm_Horizontal, symbol Diode:1N4149
- added OT5, OT6: ~, Custom:RS Pro Optical Transmitter jack, symbol Custom:RS_PRO_Optical_Transmitter_Jack
- C1: value C_drive 1uF -> 0.1uF; footprint Custom:C320C105K5R5TA -> Capacitor_THT:C_Disc_D7.0mm_W2.5mm_P5.00mm
- C19: value 0.1uF within 2mm -> 0.1uF
- C25: value 100uF UHD1H101MPD1TD -> 0.1uF optional; footprint Custom:UHD1H101MPD1TD -> Capacitor_THT:C_Disc_D7.0mm_W2.5mm_P5.00mm
- C28: value 1uF -> 10uF
Connections:
- net +10V: now also C58.1, C59.2, C60.1, L4.1, RV3.1, U10.3 (VCC), U11.3 (VCC), C65.2, C67.2, D12.2 (A)
- net +3V3: now also C1.1, C48.1, C49.1, C51.2, L2.1, RV1.1, U10.9 (VDD), U11.9 (VDD), C45.1, C61.1, C62.1, C63.1, OT5.2 (Vcc), OT6.2 (Vcc); no longer C25.1
- net Earth: now also C1.2, U10.2 (COM), U12.3 (GND), U12.4 (GND), U12.51 (GND), U12.52 (GND), C45.2, C61.2, C62.2, C63.2, C65.1, OT5.1 (GND), OT6.1 (GND)
- net at R16.1, R6.1: now also X1.7 (D33_a1io); no longer X1.13 (D13_a2io)
- net at J1.3 (Pin_3), J2.4 (Pin_4), R18.2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: no longer R12.1, X1.5 (D35_a1i)
- net at C15.1, OR5.1 (Vout): now also X1.6 (D32_a1io); no longer X1.8 (D25_a2io)
- net at C10.1, OR3.1 (Vout): now also X1.22 (TX2_io); no longer X1.20 (D4_a2io)
- net at R22.2, U1.2 (D), U9.3 (S): now also U11.5 (VS), U13.5, C66.1; no longer J4.1 (Pin_1)
- net at J3.1 (Pin_1): now also U13.4
- net at R20.2, U4.2 (D), U8.3 (S): now also J4.1 (Pin_1), U10.5 (VS), C64.1; no longer U13.5
- net +5V: now reaches C53.1, C54.2, C55.1, L3.1, RV2.1
- net +5V: now also U12.1 (5V), U12.2 (5V)
- net at OT4.3 (Vin): now also U12.56 (3); no longer X1.10 (D27_a2io)
- net at OT3.3 (Vin): now also X1.20 (D4_a2io); no longer X1.7 (D33_a1io)
- net at U2.1 (DB2): now also U12.44 (84)
- net at U2.13 (VREF_IN/OUT): now also C25.1
- net at U2.16 (DB7): now also U12.38 (74)
- net at U2.17 (DB6): now also U12.36 (72)
- net at U2.18 (DB5): now also U12.34 (70)
- net at U2.19 (DB4): now also U12.32 (68)
- net at U2.2 (DB1): now also U12.43 (85)
- net at U2.20 (DB3): now also U12.28 (64)
- net at U2.3 (DB0): now also U12.41 (83)
- net at U2.4 (!CONVST): now also U12.37 (75)
- net at U2.5 (!CS): now also U12.35 (73)
- net at U2.6 (!RD): now also U12.33 (71)
- net at U2.8 (!EOC): now also U12.31 (69)
- net at U2.9 (!PD): now also U12.25 (60)
- net at C7.1, OR2.1 (Vout): now also U12.57 (2); no longer X1.23 (D5_a2io)
- net at U11.1 (LO): now also R2.1
- net at U11.2 (COM): now also C67.1
- net at U11.6 (VB): now also C66.2, D13.1 (K)
- net at U11.7 (HO): now also R21.1
- net at C17.1, OR6.1 (Vout): now also U12.59 (144); no longer X1.9 (D26_a2io)
- net at U12.58 (1): now also OT5.3 (Vin)
- net at U12.60 (143): now also OT6.3 (Vin)
- net at U12.61 (142): now also C12.1, OR4.1 (Vout)
- net at U10.6 (VB): now also C64.2, D12.1 (K)
- net at D2.2 (A), D8.1 (K): now also U13.3; no longer U13.1
- net at D1.2 (A), D7.1 (K): now also U13.1; no longer U13.3
- net at OT2.3 (Vin): now also X1.23 (D5_a2io); no longer X1.22 (TX2_io)
- new net: R12.1, X1.5 (D35_a1i)
Other:
- note added: "High Speed Receivers"
- note added: "High Speed Transmitters"
- note added: "Slow Abstract Coms 1"
- note added: "Slow Abstract Coms 2"
- note added: "Slow Abstract Coms 3"
- note removed: "First Stage Voltage Feedback"
- note removed: "Optical Peripherals Interface"
- note removed: "Output Current Feedback"
- note removed: "Output Voltage Feedback"
- moved on the sheet: C14, C15, C16, C19, C26, C27, C28, C47, C48, C49, C50, C51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

Commit message: Gate driver for H-Bridge design finished
Parts:
- added C68: 0.1uF, Capacitor_THT:C_Disc_D7.0mm_W2.5mm_P5.00mm, symbol Device:C
- added C69: 10uF, Custom:C320C105K5R5TA, symbol Device:C
- C64: value ~ -> 1uF FG26X7R2A105KNT06
- C65, C67: value ~ -> 1uF
- C66: value ~ -> FG26X7R2A105KNT06
- D12, D13: value 1N4149 -> MUR420 R0
- R1, R13, R2, R21: value R_drive 5 -> 6
- R14, R20, R22, R3: value R_pulldown 1000 -> 1000
- RV3: value 20K -> 30K
Connections:
- net +10V: no longer C58.1, C59.2, C60.1, C65.2, C67.2, D12.2 (A), L4.1, RV3.1, U10.3 (VCC), U11.3 (VCC)
- net Earth: now also C68.2, C69.2
- net +15V: now reaches D13.2 (A)
- net +15V: now also C58.1, C59.2, C60.1, C65.2, C67.2, D12.2 (A), L4.1, RV3.1, U10.3 (VCC), U11.3 (VCC), C68.1, C69.1
Other:
- note added: "Gate Driver 9-~20v regulator"
- note removed: "10V Regulator"

Commit message: Not far from done with parts list for v2 of HVPSController
Parts:
- removed C2, C3: 1000uF UPW1E102MHD, Custom:UPW1E102MHD, symbol Device:C_Polarized
- removed C24: 0.1uF low ESR Ceramic, Capacitor_THT:C_Rect_L7.0mm_W2.5mm_P5.00mm, symbol Device:C
- removed C46: ~, Capacitor_THT:C_Rect_L7.0mm_W2.5mm_P5.00mm, symbol Custom:C322C104J5R5TA
- removed C68: 0.1uF, Capacitor_THT:C_Disc_D7.0mm_W2.5mm_P5.00mm, symbol Device:C
- removed C69: 10uF, Custom:C320C105K5R5TA, symbol Device:C
- removed D3: ~, Diode_THT:D_DO-35_SOD27_P7.62mm_Horizontal, symbol Custom:1N4619
- removed J7, J8: Conn_01x04_Pin, TerminalBlock:TerminalBlock_MaiXu_MX126-5.0-04P_1x04_P5.00mm, symbol Connector:Conn_01x04_Pin
- removed OT6: ~, Custom:RS Pro Optical Transmitter jack, symbol Custom:RS_PRO_Optical_Transmitter_Jack
- removed R15: 3K, Resistor_THT:R_Axial_DIN0207_L6.3mm_D2.5mm_P7.62mm_Horizontal, symbol Device:R
- removed U3: ~, Package_TO_SOT_THT:TO-92, symbol Custom:LM4040C25ILPR
- removed X1: ~, Custom:ESP32_WROOM-32_Dev_Board, symbol Custom:ESP32_WROOM-32_Dev_Board
- added C38: 4.7uF, Custom:C320C105K5R5TA, symbol Device:C
- added C45, C46, C64, C65: 0.1uF, Capacitor_THT:C_Disc_D7.0mm_W2.5mm_P5.00mm, symbol Device:C
- added C47, C66: 10uF, Custom:C320C105K5R5TA, symbol Device:C
- added C53, C60, C61, C75, C76: C, symbol Device:C
- added D12, D6: 1N4149, Diode_THT:D_DO-35_SOD27_P7.62mm_Horizontal, symbol Diode:1N4149
- added D16: 1N4148, Diode_THT:D_DO-35_SOD27_P7.62mm_Horizontal, symbol Diode:1N4148
- added D4: BZX55C3V0-TR, symbol Device:D_Zener
- added J10, J16: Tap debug pin, Custom:ContactViaM3, symbol Connector:Conn_01x01_Pin
- added J15, J9: Tap, Custom:ContactViaM3, symbol Connector:Conn_01x01_Pin
- added J17: Conn_01x02_Pin, symbol Connector:Conn_01x02_Pin
- added J18, J19: ~, Custom:ContactViaM3, symbol Connector:Conn_01x01_Pin
- added J24, J26: Standoff Hole, Custom:ContactViaM3, symbol Connector:Conn_01x01_Pin
- added J3, J7: ~, symbol Custom:JTAG_Header
- added K3: ~, symbol Custom:SRD-5VDC-SL-C
- added R10, R9: Pullup, Resistor_THT:R_Axial_DIN0207_L6.3mm_D2.5mm_P7.62mm_Horizontal, symbol Device:R
- added R11, R14, R28: 1K, Resistor_THT:R_Axial_DIN0207_L6.3mm_D2.5mm_P7.62mm_Horizontal, symbol Device:R
- added R13: 120K, symbol Device:R
- added R17: 50, symbol Device:R
- added R25, R26, R32, R33: R, symbol Device:R
- added R27: 22K, symbol Device:R
- added R29: 10K, Resistor_THT:R_Axial_DIN0207_L6.3mm_D2.5mm_P7.62mm_Horizontal, symbol Device:R_Small
- added RV4: 10K (adjust to 5K), symbol Device:R_Potentiometer
- added RV5: 5K (adjusted to 1.38 for 23.8K total, symbol Device:R_Potentiometer
- added S1: ~, Custom:SLW-1678105-6A-N-D, symbol Custom:SLW-1678105-6A-N-D
- added U10, U11, U13, U14, U15, U16, U8, U9: ~, symbol Custom:WS2812D
- added U18, U4, U7: ~, symbol Custom:LM4040A20I
- added U2: ~, Custom:ESP32_WROOM-32_Dev_Board, symbol Custom:ESP32_WROOM-32_Dev_Board
- added U20, U5: ~, symbol Custom:AD7822
- added U25: ~, Package_TO_SOT_THT:TO-92, symbol Custom:2N7000
- C41: renamed from C26; value 470uF -> 1000F
- C49: renamed from C50; value 470uF -> 1000uF
- C54: renamed from C25; value 0.1uF optional -> 0.1uF
- C58: renamed from C56; value 470uF -> 1000uF
- R18: value Pullup -> 100; footprint Resistor_THT:R_Axial_DIN0207_L6.3mm_D2.5mm_P7.62mm_Horizontal -> (none)
- R19: value Pullup -> 1K
- R3: renamed from R7; value R_pfb_H 270K -> 33k
- R4: renamed from R12; value R_pfb_i 1K -> 1K
- R6: renamed from R8; value R_pfb_ 10K -> 2k
- renumbered C20 to C1, C34 to C10, C6 to C11, C10 to C12, C15 to C13, C12 to C14, C17 to C15, C7 to C16, C5 to C17, C11 to C18, C16 to C19, C21 to C2, C13 to C20, C18 to C21, C8 to C22, C4 to C23, C9 to C24, C14 to C25, C27 to C26, C45 to C27, C35 to C28, C36 to C29, C22 to C3, C37 to C30, C38 to C31, C39 to C32, C40 to C33, C41 to C34, C42 to C35, C43 to C36, C44 to C37, C23 to C4, C51 to C40, C47 to C42, C48 to C43, C49 to C44, C54 to C48, C29 to C5, C52 to C50, C53 to C51, C55 to C52, C19 to C55, C28 to C56, C59 to C57, C57 to C59, C30 to C6, C58 to C62, C60 to C63, C64 to C67, C66 to C68, C61 to C69, C31 to C7, C62 to C70, C1 to C71, C63 to C72, C65 to C73, C67 to C74, C32 to C8, C33 to C9, D6 to D1, D8 to D11, D11 to D13, D12 to D14, D13 to D15, D5 to D2, D4 to D3, D9 to D5, D1 to D7, D2 to D8, D7 to D9, H5 to H1, H1 to H3, H3 to H4, J5 to J1, J10 to J11, J9 to J12, J3 to J13, J4 to J14, J6 to J2, J11 to J20, J15 to J21, J12 to J22, J13 to J23, J14 to J25, J2 to J4, J1 to J8, U7 to K1, U6 to K2, OR3 to OR2, OR5 to OR3, OR6 to OR5, OR2 to OR6, R4 to R1, R10 to R12, R11 to R15, R9 to R16, R17 to R2, R23 to R20, R13 to R21, R21 to R22, R20 to R23, R22 to R24, R1 to R30, R2 to R31, R14 to R34, R3 to R35, R16 to R5, R5 to R7, R6 to R8, S1 to S2, U13 to T1, U5 to U1, U2 to U12, U12 to U17, U16 to U19, U8 to U21, U9 to U22, U10 to U23, U11 to U24, U4 to U26, U1 to U27, U14 to U3, U15 to U6
Connections:
- net +36V: now also C60.1, C61.1
- net +3V3: now also C46.1, C47.1, C65.1, C66.1, R10.1, R11.1, R14.1, R17.1, R9.1, U20.14 (VDD), U5.14 (VDD); no longer R18.1
- net +5V: now also D16.1 (K), K3.2, K3.3, S1.5, U10.2 (VDD), U11.2 (VDD), U13.2 (VDD), U14.2 (VDD), U15.2 (VDD), U16.2 (VDD), U8.2 (VDD), U9.2 (VDD); no longer U17.1 (5V), U17.2 (5V)
- net Earth: now also C15.1, OR5.1 (Vout), R18.2, U17.47 (GND), U17.48 (GND), U17.59 (144), U17.95 (GND), U17.96 (GND), U23.13 (VSS), U24.13 (VSS), C38.2, C45.2, C46.2, C47.2, C53.2, C64.2, C65.2, C66.2, D4.2 (A), J17.2 (Pin_2), J24.1 (Pin_1), J26.1 (Pin_1), J3.10 (GND), J3.2 (GND), J7.10 (GND), J7.2 (GND), R29.2, R32.2, R33.2, RV4.2, RV5.2, U10.3 (GND), U11.3 (GND), U13.3 (GND), U14.3 (GND), U15.3 (GND), U16.3 (GND), U18.3 (Anode), U2.14 (GND), U2.17 (GND), U20.15 (AGND), U20.7 (DGND), U25.1 (S), U4.3 (Anode), U5.15 (AGND), U5.7 (DGND), U7.3 (Anode), U8.3 (GND), U9.3 (GND)
- net at S2.6: now also U2.16 (3V3)
- net at R5.1, R8.1: now also U2.6 (D32_a1io)
- net at C12.1, OR2.1 (Vout): now also U2.2 (VP_a1i)
- net at C11.1, OR1.1 (Vout): now also U2.3 (VN_a1i)
- net at R4.1: now also U2.5 (D35_a1i)
- net at R3.2, R4.2, R6.1: now also C38.1, D4.1 (K)
- net at C13.1, OR3.1 (Vout): now also U2.30 (D23_io)
- net at C54.1, U12.13 (VREF_IN/OUT): now also R14.2, U7.2 (Cathode)
- net at C67.1, J14.1 (Pin_1), R23.2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: now also C75.1, J18.1 (Pin_1), R25.2
- net at J4.4 (Pin_4), J8.3 (Pin_3): now also R10.2, U2.20 (D4_a2io); no longer R18.2
- net at J4.3 (Pin_3), J8.4 (Pin_4): now also R9.2, U2.22 (TX2_io); no longer R19.2
- net at OT3.3 (Vin): now also U2.23 (D5_a2io)
- net at U17.60 (143): now also U5.20 (DB3)
- net at U12.1 (DB2): now also U17.38 (74); no longer U17.44 (84)
- net at U12.16 (DB7): now also U17.36 (72); no longer U17.38 (74)
- net at U12.17 (DB6): now also U17.34 (70); no longer U17.36 (72)
- net at U12.18 (DB5): now also U17.32 (68); no longer U17.34 (70)
- net at U12.19 (DB4): now also U17.28 (64); no longer U17.32 (68)
- net at U12.2 (DB1): now also U17.44 (84); no longer U17.43 (85)
- net at U12.20 (DB3): now also U17.26 (59); no longer U17.28 (64)
- net at U12.3 (DB0): now also U17.43 (85); no longer U17.41 (83)
- net at U12.4 (!CONVST): now also U17.41 (83); no longer U17.37 (75)
- net at U12.5 (!CS): now also U17.37 (75); no longer U17.35 (73)
- net at U12.6 (!RD): now also U17.35 (73); no longer U17.33 (71)
- net at U12.8 (!EOC): now also U17.33 (71); no longer U17.31 (69)
- net at U12.9 (!PD): now also U17.81 (112), U20.9 (!PD), U5.9 (!PD); no longer U17.25 (60)
- net at OT1.3 (Vin): now also U2.25 (D19_io)
- net at C68.1, R24.2, T1.5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: now also C76.1, J19.1 (Pin_1), R26.2
- net at U24.10 (HIN): now also U17.31 (69), U23.12 (LIN)
- net at U24.11 (SD): now also U17.83 (110), U23.11 (SD)
- net at U24.12 (LIN): now also U17.25 (60), U23.10 (HIN)
- net at U17.11 (39): now also U2.29 (D22_io)
- net at U17.12 (38): now also U20.1 (DB2)
- net at U17.13 (43): now also U2.13 (D13_a2io)
- net at U17.14 (42): now also U20.2 (DB1)
- net at U17.16 (44): now also U20.3 (DB0)
- net at U17.17 (50): now also U2.11 (D14_a2io)
- net at U17.18 (49): now also U20.4 (!CONVST)
- net at U17.19 (52): now also U2.10 (D27_a2io)
- net at U17.20 (51): now also U20.5 (!CS)
- net at U17.21 (54): now also U2.9 (D26_a2io)
- net at U17.22 (53): now also U20.6 (!RD)
- net at U17.23 (58): now also U2.4 (D34_a1i)
- net at U17.24 (55): now also U20.8 (!EOC)
- net at U17.5 (30): now also U2.26 (D21_io)
- net at U17.6 (28): now also U20.16 (DB7)
- net at U17.62 (141): now also U5.19 (DB4)
- net at U17.66 (135): now also U5.18 (DB5)
- net at U17.69 (129): now also U20.17 (DB6)
- net at U17.70 (128): now also U5.17 (DB6)
- net at U17.71 (127): now also U20.18 (DB5)
- net at U17.72 (126): now also U5.16 (DB7)
- net at U17.73 (125): now also U20.19 (DB4)
- net at U17.74 (124): now also U5.1 (DB2)
- net at U17.75 (121): now also U20.20 (DB3)
- net at U17.76 (120): now also U5.2 (DB1)
- net at U17.80 (113): now also U5.3 (DB0)
- net at U17.82 (111): now also U5.4 (!CONVST)
- net at U17.84 (106): now also U5.5 (!CS)
- net at U17.86 (104): now also U5.6 (!RD)
- net at U17.89 (100): now also U5.8 (!EOC)
- net at OT2.3 (Vin): now also U2.24 (D18_io)
- new net: R13.2, RV4.1
- new net: C75.2, R32.1
- new net: D12.2 (A), J15.1 (Pin_1), J16.1 (Pin_1), R27.1, U20.11 (VIN1)
- new net: C64.1, R19.2, U18.2 (Cathode), U20.13 (VREF_IN/OUT)
- new net: C60.2, R25.1
- new net: D6.2 (A), J10.1 (Pin_1), J9.1 (Pin_1), R13.1, U5.11 (VIN1)
- new net: U10.1 (DOUT), U9.4 (DIN)
- new net: U10.4 (DIN), U11.1 (DOUT)
- new net: C61.2, R26.1
- new net: J3.1 (TCK), J7.1 (TCK)
- new net: J3.3 (TDO), J7.3 (TDO)
- new net: J3.4 (VCC), S1.2
- new net: J3.5 (TMS), J7.5 (TMS)
- new net: J3.6 (NC), J7.6 (NC)
- new net: J3.7 (NC), J7.7 (NC)
- new net: J3.8 (NC), J7.8 (NC)
- new net: J3.9 (TDI), J7.9 (TDI)
- new net: D16.2 (A), K3.1, U25.3 (D)
- new net: J17.1 (Pin_1), K3.4
- new net: R28.2, U25.2 (G)
- new net: U11.4 (DIN), U2.7 (D33_a1io)
- new net: R28.1, R29.1, U2.8 (D25_a2io)
- new net: U13.4 (DIN), U14.1 (DOUT)
- new net: C45.1, R11.2, U4.2 (Cathode), U5.13 (VREF_IN/OUT)
- new net: C76.2, R33.1
- new net: U16.4 (DIN), U8.1 (DOUT)
- new net: U8.4 (DIN), U9.1 (DOUT)
- new net: R27.2, RV5.1
- new net: U14.4 (DIN), U15.1 (DOUT)
- new net: C53.1, D12.1 (K), D6.1 (K), R17.2, R18.1
- new net: U15.4 (DIN), U16.1 (DOUT)
- new net: S1.6, U17.1 (5V), U17.2 (5V)
- new net: J7.4 (VCC), S1.1
Other:
- note added: "Fan Drive"
- note added: "Ionic wind arrestor 20mA"
- note added: "LED Status Indicator"
- note added: "Voltage Feedback 1 (First Stage)"
- note added: "Voltage Feedback 2 (Output)"
- note removed: "2.5V Reference"
- moved on the sheet: C14, C15, C16, C20, C21, C22, C26, C27, C54, C55, C56, C67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

Commit message: Started on the verilog and fpga :)
Parts:
- added H5, H6, H7: Heatsink, Custom:647-25ABEP, symbol Connector:Conn_01x01_Pin
- H1, H2, H3, H4: value Heatsink 5 -> Heatsink
- R21, R22, R30, R31: value 6 -> 6.2
Connections:
- net Earth: now also H5.1 (Pin_1), H6.1 (Pin_1), H7.1 (Pin_1)

Commit message: having a hard time pulling myself away from this. Must stop now.
Parts:
- removed H5, H6, H7: Heatsink, Custom:647-25ABEP, symbol Connector:Conn_01x01_Pin
- removed J3, J7: ~, symbol Custom:JTAG_Header
- removed S1: ~, Custom:SLW-1678105-6A-N-D, symbol Custom:SLW-1678105-6A-N-D
- added J3, J5, J6: ~, Connector_PinHeader_2.54mm:PinHeader_1x01_P2.54mm_Vertical, symbol Connector:Conn_01x01_Pin
- added L5, L6, L7: ~, Custom:5026 Inductor, symbol Device:L
- added R36, R37: 4.7, Resistor_THT:R_Axial_DIN0207_L6.3mm_D2.5mm_P5.08mm_Vertical, symbol Device:R_Small
- C38, C42, C44, C48, C50, C52, C57, C59, C63: footprint Custom:C320C105K5R5TA -> Capacitor_THT:C_Rect_L7.0mm_W2.5mm_P5.00mm
- C40, C47, C56, C66, C70, C72: footprint Custom:C320C105K5R5TA -> Capacitor_THT:C_Rect_L4.0mm_W2.5mm_P2.50mm
- C41: value 1000F -> 1000uF; footprint (none) -> Custom:ECA-1JM102
- C43, C51, C62: footprint (none) -> Custom:UPW1E471MPD6TA
- C45, C46, C54, C55, C64, C65, C69, C71: footprint Capacitor_THT:C_Disc_D7.0mm_W2.5mm_P5.00mm -> Capacitor_THT:C_Rect_L7.0mm_W2.5mm_P5.00mm
- C49, C58: footprint (none) -> Custom:ECA-1JM102
- C53: footprint (none) -> Capacitor_THT:C_Rect_L7.0mm_W2.5mm_P5.00mm
- C67, C68, C73, C74: footprint Custom:C320C105K5R5TA -> Capacitor_THT:C_Rect_L7.0mm_W2.0mm_P5.00mm
- D1, D11, D12, D16, D2, D3, D6, D7, D8, D9: footprint Diode_THT:D_DO-35_SOD27_P7.62mm_Horizontal -> Diode_THT:D_DO-35_SOD27_P10.16mm_Horizontal
- D10, D13, D5: footprint Diode_THT:D_DO-201AD_P15.24mm_Horizontal -> Diode_THT:D_DO-201AD_P12.70mm_Horizontal
- D14: value MUR420 R0 -> MUR220RLG; footprint Diode_THT:D_DO-35_SOD27_P7.62mm_Horizontal -> Diode_THT:D_DO-41_SOD81_P5.08mm_Vertical_AnodeUp
- D15: footprint Diode_THT:D_DO-35_SOD27_P7.62mm_Horizontal -> Diode_THT:D_DO-41_SOD81_P7.62mm_Horizontal
- D4: footprint (none) -> Diode_THT:D_DO-35_SOD27_P10.16mm_Horizontal
- J1, J13, J14, J2: footprint Custom:5055556-9 -> Custom:PCB-3 (M4)
- J10, J16, J18, J19: footprint Custom:ContactViaM3 -> Connector_PinHeader_2.54mm:PinHeader_1x01_P2.54mm_Vertical
- J15, J9: footprint Custom:ContactViaM3 -> Custom:PCB-1 (M4)
- J17: footprint (none) -> Connector_JST:JST_XH_B2B-XH-A_1x02_P2.50mm_Vertical
- K3: footprint (none) -> Custom:SRD-5VDC-SL-C
- L2, L3, L4: footprint (none) -> Custom:5026 Inductor
- R12, R13, R15, R17, R18, R20, R27: footprint (none) -> Resistor_THT:R_Axial_DIN0207_L6.3mm_D2.5mm_P7.62mm_Horizontal
- R16: footprint (none) -> Custom:SL2TTED10R0F
- R2, R7: footprint Resistor_THT:R_Axial_DIN0309_L9.0mm_D3.2mm_P12.70mm_Horizontal -> Resistor_THT:R_Axial_DIN0207_L6.3mm_D2.5mm_P7.62mm_Horizontal
- R21, R30, R31: footprint Resistor_THT:R_Axial_DIN0207_L6.3mm_D2.5mm_P10.16mm_Horizontal -> Resistor_THT:R_Axial_DIN0207_L6.3mm_D2.5mm_P7.62mm_Horizontal
- R23, R24: footprint Resistor_THT:R_Axial_DIN0207_L6.3mm_D2.5mm_P7.62mm_Horizontal -> Resistor_THT:R_Axial_DIN0207_L6.3mm_D2.5mm_P5.08mm_Vertical
- RV1, RV2, RV3, RV4, RV5: footprint (none) -> Potentiometer_THT:Potentiometer_Bourns_3296W_Vertical
- T1: footprint (none) -> Custom:CST2020-200L
- U10, U11, U13, U14, U15, U16, U8, U9: footprint (none) -> LED_THT:LED_D5.0mm-4_RGB_Wide_Pins
- U12, U20, U5: footprint (none) -> Package_DIP:DIP-20_W7.62mm_Socket_LongPads
- U17: footprint (none) -> Custom:EP4CE6E22C8N_FPGA_Development_Board_
- U18, U4, U7: footprint (none) -> Package_TO_SOT_THT:TO-92
- U19, U3, U6: footprint (none) -> Package_TO_SOT_THT:TO-220-5_Vertical
- U21, U22, U26, U27: footprint Custom:IXFP60N25X3 -> Custom:IXFP60N25X3_2
- U23, U24: footprint (none) -> Package_DIP:DIP-14_W7.62mm_Socket_LongPads
Connections:
- net +15V: now also J6.1 (Pin_1), R36.1, R37.1; no longer D14.2 (A), D15.2 (A)
- net +36V: now also H1.1 (Pin_1), H2.1 (Pin_1), L5.1, L6.1, L7.1; no longer C41.1, C42.1, C49.1, C50.1, C58.1, C59.1, U19.1 (VIN), U3.1 (VIN), U6.1 (VIN)
- net +3V3: now also J3.1 (Pin_1)
- net +5V: now also U17.1 (5V), U17.2 (5V), J5.1 (Pin_1)
- net Earth: no longer C15.1, H1.1 (Pin_1), H2.1 (Pin_1), H3.1 (Pin_1), H4.1 (Pin_1), OR5.1 (Vout), U17.59 (144)
- net at C14.1, OR4.1 (Vout): now also U17.13 (43); no longer U17.61 (142)
- net at R5.1, R8.1: now also U2.26 (D21_io); no longer U2.6 (D32_a1io)
- net at C67.1, C75.1, J18.1 (Pin_1)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: now also H3.1 (Pin_1), J13.1 (Pin_1); no longer J14.1 (Pin_1)
- net at U20.1 (DB2): now also U17.14 (42); no longer U17.12 (38)
- net at U20.16 (DB7): now also U17.71 (127); no longer U17.6 (28)
- net at U20.18 (DB5): now also U17.61 (142); no longer U17.71 (127)
- net at U20.19 (DB4): now also U17.59 (144); no longer U17.73 (125)
- net at U20.2 (DB1): now also U17.12 (38); no longer U17.14 (42)
- net at U20.20 (DB3): now also U17.57 (2); no longer U17.75 (121)
- net at U20.3 (DB0): now also U17.6 (28); no longer U17.16 (44)
- net at U20.4 (!CONVST): now also U17.16 (44); no longer U17.18 (49)
- net at U20.5 (!CS): now also U17.18 (49); no longer U17.20 (51)
- net at U20.6 (!RD): now also U17.20 (51); no longer U17.22 (53)
- net at U20.8 (!EOC): now also U17.22 (53); no longer U17.24 (55)
- net at U12.9 (!PD), U20.9 (!PD), U5.9 (!PD): now also U17.33 (71); no longer U17.81 (112)
- net at T1.4: now also J14.1 (Pin_1); no longer J13.1 (Pin_1)
- net at U2.10 (D27_a2io): now also U17.21 (54); no longer U17.19 (52)
- net at U2.11 (D14_a2io): now also U17.19 (52); no longer U17.17 (50)
- net at U2.13 (D13_a2io): now also U17.17 (50); no longer U17.13 (43)
- net at U17.5 (30): now also C16.1, OR6.1 (Vout); no longer U2.26 (D21_io)
- net at U17.11 (39): now also C15.1, OR5.1 (Vout); no longer U2.29 (D22_io)
- net at U2.4 (D34_a1i): now also U17.31 (69); no longer U17.23 (58)
- net at U11.4 (DIN): now also U2.6 (D32_a1io); no longer U2.7 (D33_a1io)
- net at R28.1, R29.1: now also U2.7 (D33_a1io); no longer U2.8 (D25_a2io)
- net at U2.9 (D26_a2io): now also U17.23 (58); no longer U17.21 (54)
- net at C68.1, C76.1, J19.1 (Pin_1)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: now also H4.1 (Pin_1)
- net at U12.1 (DB2): now also U17.86 (104); no longer U17.38 (74)
- net at U12.16 (DB7): now also U17.70 (128); no longer U17.36 (72)
- net at U12.17 (DB6): now also U17.72 (126); no longer U17.34 (70)
- net at U12.18 (DB5): now also U17.74 (124); no longer U17.32 (68)
- net at U12.19 (DB4): now also U17.76 (120); no longer U17.28 (64)
- net at U12.2 (DB1): now also U17.84 (106); no longer U17.44 (84)
- net at U12.20 (DB3): now also U17.80 (113); no longer U17.26 (59)
- net at U12.3 (DB0): now also U17.82 (111); no longer U17.43 (85)
- net at U12.4 (!CONVST): now also U17.83 (110); no longer U17.41 (83)
- net at U12.5 (!CS): now also U17.81 (112); no longer U17.37 (75)
- net at U12.6 (!RD): now also U17.75 (121); no longer U17.35 (73)
- net at U12.8 (!EOC): now also U17.73 (125); no longer U17.33 (71)
- net at U23.12 (LIN), U24.10 (HIN): now also U17.62 (141); no longer U17.31 (69)
- net at U23.11 (SD), U24.11 (SD): now also U17.60 (143); no longer U17.83 (110)
- net at U23.10 (HIN), U24.12 (LIN): now also U17.66 (135); no longer U17.25 (60)
- net at U5.20 (DB3): now also U17.34 (70); no longer U17.60 (143)
- net at U5.19 (DB4): now also U17.32 (68); no longer U17.62 (141)
- net at U5.18 (DB5): now also U17.28 (64); no longer U17.66 (135)
- net at U5.17 (DB6): now also U17.26 (59); no longer U17.70 (128)
- net at U5.16 (DB7): now also U17.24 (55); no longer U17.72 (126)
- net at U5.1 (DB2): now also U17.44 (84); no longer U17.74 (124)
- net at U5.2 (DB1): now also U17.38 (74); no longer U17.76 (120)
- net at U5.3 (DB0): now also U17.36 (72); no longer U17.80 (113)
- net at U5.4 (!CONVST): now also U17.43 (85); no longer U17.82 (111)
- net at U5.5 (!CS): now also U17.41 (83); no longer U17.84 (106)
- net at U5.6 (!RD): now also U17.37 (75); no longer U17.86 (104)
- net at U17.89 (100): now also U2.29 (D22_io); no longer U5.8 (!EOC)
- new net: C58.1, C59.1, L7.2, U19.1 (VIN)
- new net: C49.1, C50.1, L6.2, U6.1 (VIN)
- new net: C41.1, C42.1, L5.2, U3.1 (VIN)
- new net: U17.25 (60), U2.8 (D25_a2io)
- new net: D14.2 (A), R36.2
- new net: D15.2 (A), R37.2
- new net: U17.35 (73), U5.8 (!EOC)
Other:
- moved on the sheet: C45, C46, C47, C53, C54, C55, C56, C60, C61, C64, C65, C66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

Commit message: PCB coming together :)
Parts:
- added C39: 1000uF, Custom:ECA-1JM102, symbol Device:C_Polarized
- added C77, C80, C81, C82: 0.1uF, Capacitor_THT:C_Rect_L7.0mm_W2.5mm_P5.00mm, symbol Device:C
- added C78: 470uF, Custom:UPW1E471MPD6TA, symbol Device:C_Polarized
- added C79: 2.2nF, Capacitor_THT:C_Rect_L7.0mm_W2.5mm_P5.00mm, symbol Device:C
- added D17: 1N5822, Diode_THT:D_DO-201AD_P12.70mm_Horizontal, symbol Diode:1N5822
- added J7: ~, Connector_PinHeader_2.54mm:PinHeader_1x01_P2.54mm_Vertical, symbol Connector:Conn_01x01_Pin
- added L8: ~, Custom:5026 Inductor, symbol Device:L
- added L9: 68uH, Custom:5026 Inductor, symbol Device:L
- added R38: 2K 1%, Resistor_THT:R_Axial_DIN0207_L6.3mm_D2.5mm_P7.62mm_Horizontal, symbol Device:R
- added RV6: 30K, Potentiometer_THT:Potentiometer_Bourns_3296W_Vertical, symbol Device:R_Potentiometer
- added U28, U29, U30, U31: ~, Custom:HW-677 LM2596HVS DC-DC, symbol Custom:HW-677_LM2596HVS_DC-DC
- added U32: ~, Package_TO_SOT_THT:TO-220-5_Vertical, symbol Custom:LM2596HV
- R21, R22, R30, R31: value 6.2 -> 4.7
Connections:
- net +15V: now also U30.4 (OUT+); no longer R37.1
- net +36V: now also L8.1
- net +3V3: now also U28.4 (OUT+)
- net +5V: now also U29.4 (OUT+)
- net Earth: now also C39.2, C77.2, C78.2, C80.2, C81.2, C82.2, D17.2 (A), R38.2, U28.2 (IN-), U28.3 (OUT-), U29.2 (IN-), U29.3 (OUT-), U30.2 (IN-), U30.3 (OUT-), U31.2 (IN-), U31.3 (OUT-), U32.3 (GND), U32.5 (ON/OFF)
- net at C58.1, C59.1, L7.2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: now also U30.1 (IN+)
- net at C49.1, C50.1, L6.2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: now also U29.1 (IN+)
- net at C41.1, C42.1, L5.2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: now also U28.1 (IN+)
- net at D12.2 (A), J15.1 (Pin_1), J16.1 (Pin_1)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: now also C82.1
- net at D6.2 (A), J10.1 (Pin_1), J9.1 (Pin_1)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: now also C81.1
- net at U23.12 (LIN), U24.10 (HIN): now also U17.66 (135); no longer U17.62 (141)
- net at U23.11 (SD), U24.11 (SD): now also U17.62 (141); no longer U17.60 (143)
- net at U23.10 (HIN), U24.12 (LIN): now also U17.60 (143); no longer U17.66 (135)
- new net: C39.1, C77.1, L8.2, U31.1 (IN+), U32.1 (VIN)
- new net: D17.1 (K), L9.2, U32.2 (OUTPUT)
- new net: C79.1, R38.1, RV6.2, U32.4 (FEEDBACK)
- new net +14V: C78.1, C79.2, C80.1, J7.1 (Pin_1), L9.1, R37.1, RV6.1, U31.4 (OUT+)
Other:
- moved on the sheet: C40, C41, C42, C43, C44, C45, C46, C47, C48, C49, C50, C51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
