File: Kicad/HVPSController2/HVPSController2.kicad_sch (KiCad schematic)
At the start: 231 parts, among them J1 Vsupply, J10 Tap debug pin, J11 USB RWGBS, J12 USB RWGBS, J13 Conn_01x01_Pin, J14 Conn_01x01_Pin, J15 Tap, J16 Tap debug pin, J17 Conn_01x02_Pin, J2 GND, J20 Standoff Hole, J21 Standoff Hole, J22 Standoff Hole, J23 Standoff Hole, J24 Standoff Hole, J25 Standoff Hole, J26 Standoff Hole, J4 Conn_01x08_Pin, J8 SCL, SDA, +, GND, J9 Tap

Commit message: Going great.
Parts:
- D1, D2, D3: footprint Diode_THT:D_DO-35_SOD27_P10.16mm_Horizontal -> Diode_THT:D_DO-35_SOD27_P7.62mm_Horizontal
- D12, D6: footprint Diode_THT:D_DO-35_SOD27_P10.16mm_Horizontal -> Diode_THT:D_DO-35_SOD27_P5.08mm_Vertical_AnodeUp
Connections:
- net +14V: now also C74.2, U24.3 (VCC)
- net +15V: no longer C74.2, U24.3 (VCC)
- net Earth: now also U12.5 (!CS), U20.5 (!CS), U5.5 (!CS)
- net at S2.1: now also J11.1 (Pin_1); no longer J12.1 (Pin_1)
- net at S2.2: now also J12.1 (Pin_1); no longer J11.1 (Pin_1)
- net at R5.1, U2.26 (D21_io): no longer R8.1
- net at R5.2, U1.2 (G): now also R8.1
- net at U20.16 (DB7): now also U17.75 (121); no longer U17.71 (127)
- net at U20.17 (DB6): now also U17.73 (125); no longer U17.69 (129)
- net at U20.18 (DB5): now also U17.71 (127); no longer U17.61 (142)
- net at U20.19 (DB4): now also U17.69 (129); no longer U17.59 (144)
- net at U20.2 (DB1): now also U17.16 (44); no longer U17.12 (38)
- net at U20.20 (DB3): now also U17.61 (142); no longer U17.57 (2)
- net at U20.3 (DB0): now also U17.18 (49); no longer U17.6 (28)
- net at U20.4 (!CONVST): now also U17.20 (51); no longer U17.16 (44)
- net at U20.6 (!RD): now also U17.22 (53); no longer U17.20 (51)
- net at U20.8 (!EOC): now also U17.24 (55); no longer U17.22 (53)
- net at OT4.3 (Vin): now also U17.6 (28); no longer U17.56 (3)
- net at R28.2, U25.2 (G): now also R29.1
- net at R28.1, U2.7 (D33_a1io): no longer R29.1
- net at U12.1 (DB2): now also U17.72 (126); no longer U17.86 (104)
- net at U12.17 (DB6): now also U17.66 (135); no longer U17.72 (126)
- net at U12.18 (DB5): now also U17.62 (141); no longer U17.74 (124)
- net at U12.19 (DB4): now also U17.60 (143); no longer U17.76 (120)
- net at U12.2 (DB1): now also U17.74 (124); no longer U17.84 (106)
- net at U12.20 (DB3): now also U17.58 (1); no longer U17.80 (113)
- net at U12.3 (DB0): now also U17.76 (120); no longer U17.82 (111)
- net at U12.4 (!CONVST): now also U17.80 (113); no longer U17.83 (110)
- net at U17.81 (112): now also U24.10 (HIN); no longer U12.5 (!CS)
- net at U12.6 (!RD): now also U17.82 (111); no longer U17.75 (121)
- net at U12.8 (!EOC): now also U17.84 (106); no longer U17.73 (125)
- net at OT5.3 (Vin): now also U17.12 (38); no longer U17.58 (1)
- net at U5.16 (DB7): now also U17.26 (59); no longer U17.24 (55)
- net at U5.17 (DB6): now also U17.28 (64); no longer U17.26 (59)
- net at U5.18 (DB5): now also U17.32 (68); no longer U17.28 (64)
- net at U5.19 (DB4): now also U17.34 (70); no longer U17.32 (68)
- net at U5.20 (DB3): now also U17.36 (72); no longer U17.34 (70)
- net at U5.3 (DB0): now also U17.38 (74); no longer U17.36 (72)
- net at U5.2 (DB1): now also U17.44 (84); no longer U17.38 (74)
- net at U17.41 (83): now also U5.4 (!CONVST); no longer U5.5 (!CS)
- net at U17.43 (85): now also U5.1 (DB2); no longer U5.4 (!CONVST)
- new net: U17.83 (110), U24.11 (SD)
- new net: U17.86 (104), U24.12 (LIN)
- new net: U17.59 (144), U23.10 (HIN)
- new net: U17.57 (2), U23.11 (SD)
- new net: U17.56 (3), U23.12 (LIN)
Other:
- moved on the sheet: R16
