File: Kicad/HVPSController2/HVPSController2.kicad_sch (KiCad schematic)
At the start: 231 parts, among them J1 Vsupply, J10 Tap debug pin, J11 USB RWGBS, J12 USB RWGBS, J13 Conn_01x01_Pin, J14 Conn_01x01_Pin, J15 Tap, J16 Tap debug pin, J17 Conn_01x02_Pin, J2 GND, J20 Standoff Hole, J21 Standoff Hole, J22 Standoff Hole, J23 Standoff Hole, J24 Standoff Hole, J25 Standoff Hole, J26 Standoff Hole, J4 Conn_01x08_Pin, J8 SCL, SDA, +, GND, J9 Tap

Commit message: Going great.
Parts:
- removed C39, C41, C49, C58: 1000uF, Custom:ECA-1JM102, symbol Device:C_Polarized
- removed C40: 10nF, Capacitor_THT:C_Rect_L4.0mm_W2.5mm_P2.50mm, symbol Device:C
- removed C42, C44, C50, C52, C59, C63, C77, C80: 0.1uF, Capacitor_THT:C_Rect_L7.0mm_W2.5mm_P5.00mm, symbol Device:C
- removed C43, C51, C62, C78: 470uF, Custom:UPW1E471MPD6TA, symbol Device:C_Polarized
- removed C48: 4.7nF, Capacitor_THT:C_Rect_L7.0mm_W2.5mm_P5.00mm, symbol Device:C
- removed C57, C79: 2.2nF, Capacitor_THT:C_Rect_L7.0mm_W2.5mm_P5.00mm, symbol Device:C
- removed D10, D13, D17, D5: 1N5822, Diode_THT:D_DO-201AD_P12.70mm_Horizontal, symbol Diode:1N5822
- removed J3, J5, J6, J7: ~, Connector_PinHeader_2.54mm:PinHeader_1x01_P2.54mm_Vertical, symbol Connector:Conn_01x01_Pin
- removed L3, L4, L9: 68uH, Custom:5026 Inductor, symbol Device:L
- removed R12, R15, R20, R38: 2K 1%, Resistor_THT:R_Axial_DIN0207_L6.3mm_D2.5mm_P7.62mm_Horizontal, symbol Device:R
- removed RV1: 5K, Potentiometer_THT:Potentiometer_Bourns_3296W_Vertical, symbol Device:R_Potentiometer
- removed RV2: 10K, Potentiometer_THT:Potentiometer_Bourns_3296W_Vertical, symbol Device:R_Potentiometer
- removed RV3, RV6: 30K, Potentiometer_THT:Potentiometer_Bourns_3296W_Vertical, symbol Device:R_Potentiometer
- removed U13, U14, U15, U16: ~, LED_THT:LED_D5.0mm-4_RGB_Wide_Pins, symbol Custom:WS2812D
- removed U19, U3, U32, U6: ~, Package_TO_SOT_THT:TO-220-5_Vertical, symbol Custom:LM2596HV
- added U3: ~, Custom:HW-677 LM2596HVS DC-DC, symbol Custom:HW-677_LM2596HVS_DC-DC
- L2: value 68uH -> ~
Connections:
- net +36V: now also L2.1
- net +3V3: now also U3.4 (OUT+); no longer L2.1
- net Earth: now also U12.9 (!PD), U20.9 (!PD), U5.9 (!PD), U3.2 (IN-), U3.3 (OUT-); no longer R1.3 (C1), R1.4 (C2)
- net at C12.1, OR2.1 (Vout): now also U2.5 (D35_a1i); no longer U2.2 (VP_a1i)
- net at R4.1: now also U2.2 (VP_a1i); no longer U2.5 (D35_a1i)
- net at C13.1, OR3.1 (Vout): now also U2.23 (D5_a2io); no longer U2.30 (D23_io)
- net at D3.1 (K), K1.4, K2.2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: now also R1.2; no longer R1.1
- net at J4.3 (Pin_3), R9.2, U2.22 (TX2_io): now also J8.3 (Pin_3); no longer J8.4 (Pin_4)
- net at U2.10 (D27_a2io): now also U17.19 (52); no longer U17.21 (54)
- net at U2.11 (D14_a2io): now also U17.17 (50); no longer U17.19 (52)
- net at U2.13 (D13_a2io): now also J4.4 (Pin_4), J8.4 (Pin_4), R10.2; no longer U17.17 (50)
- net at OT3.3 (Vin): now also U2.24 (D18_io); no longer U2.23 (D5_a2io)
- net at OT2.3 (Vin): now also U2.25 (D19_io); no longer U2.24 (D18_io)
- net at OT1.3 (Vin): now also U2.30 (D23_io); no longer U2.25 (D19_io)
- net at U2.29 (D22_io): now also U17.33 (71); no longer U17.89 (100)
- net at U11.4 (DIN): now also U2.20 (D4_a2io); no longer U2.6 (D32_a1io)
- net at R28.1: now also U2.6 (D32_a1io); no longer U2.7 (D33_a1io)
- net at U17.25 (60): now also U2.7 (D33_a1io); no longer U2.8 (D25_a2io)
- net at U17.23 (58): now also U2.8 (D25_a2io); no longer U2.9 (D26_a2io)
- net at K2.4, L1.1: now also R1.1; no longer R1.2
- net at L2.2: now also U3.1 (IN+)
- new net: U17.21 (54), U2.9 (D26_a2io)
Other:
- moved on the sheet: R1

Commit message: Put in place emulation of the ESP32 FPGA interface in C#.
Parts:
- removed J24: Standoff Hole, Custom:ContactViaM3, symbol Connector:Conn_01x01_Pin
- R23: footprint Resistor_THT:R_Axial_DIN0207_L6.3mm_D2.5mm_P5.08mm_Vertical -> Resistor_THT:R_Axial_DIN0207_L6.3mm_D2.5mm_P7.62mm_Horizontal
Connections:
- net +3V3: no longer C20.1, C21.1, C22.1, C26.1, C27.1, C55.1, C56.1, C69.1, C70.1, J4.1 (Pin_1), J8.2 (Pin_2), OR4.3 (Vcc), OR5.3 (Vcc), OR6.3 (Vcc), OT4.2 (Vcc), OT5.2 (Vcc), R10.1, R14.1, R9.1, U12.14 (VDD), U23.9 (VDD), U3.4 (OUT+)
- net Earth: now also C74.1, U24.2 (COM)
- net +14V renamed 15V_2
- new net 3v3_2: C20.1, C21.1, C22.1, C26.1, C27.1, C55.1, C56.1, C69.1, C70.1, J4.1 (Pin_1), J8.2 (Pin_2), OR4.3 (Vcc), OR5.3 (Vcc), OR6.3 (Vcc), OT4.2 (Vcc), OT5.2 (Vcc), R10.1, R14.1, R9.1, U12.14 (VDD), U23.9 (VDD), U3.4 (OUT+)

Commit message: Board almost done got some more checks to do first been cleaning up nicely.
Parts:
- removed C60, C61, C75, C76: C, symbol Device:C
- removed R25, R26, R32, R33: R, symbol Device:R
- added J24: Conn_01x02_Pin, Connector_JST:JST_XH_B2B-XH-A_1x02_P2.50mm_Vertical, symbol Connector:Conn_01x02_Pin
- added J3, J5, J6, J7: Snubber, Custom:Snubber_Connection_1, symbol Connector:Conn_01x02_Pin
- S2: footprint Custom:SLW-1678105-6A-N-D -> Custom:MSS-04A
Connections:
- net +36V: now also J3.2 (Pin_2), J5.2 (Pin_2)
- net Earth: now also J24.2 (Pin_2), J6.1 (Pin_1), J7.1 (Pin_1)
- net at C67.1, H3.1 (Pin_1), J13.1 (Pin_1)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: now also J3.1 (Pin_1), J6.2 (Pin_2)
- net at J17.1 (Pin_1), K3.4: now also J24.1 (Pin_1)
- net at C68.1, H4.1 (Pin_1), J19.1 (Pin_1)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: now also J5.1 (Pin_1), J7.2 (Pin_2)
Other:
- moved on the sheet: R29

Commit message: Going great think im ready to order the pcb!
Parts:
- removed J10, J16: Tap debug pin, Connector_PinHeader_2.54mm:PinHeader_1x01_P2.54mm_Vertical, symbol Connector:Conn_01x01_Pin
- added J10, J16, J32, J33, J34, J35, J36: Conn_01x02_Pin, Connector_PinHeader_2.54mm:PinHeader_1x02_P2.54mm_Vertical, symbol Connector:Conn_01x02_Pin
- added J27, J28, J29, J30, J31: ~, Connector_PinHeader_2.54mm:PinHeader_1x01_P2.54mm_Vertical, symbol Connector:Conn_01x01_Pin
- R34: footprint Resistor_THT:R_Axial_DIN0207_L6.3mm_D2.5mm_P7.62mm_Horizontal -> Resistor_THT:R_Axial_DIN0207_L6.3mm_D2.5mm_P5.08mm_Vertical
Connections:
- net +15V: now also J35.1 (Pin_1)
- net +3V3: now also U20.9 (!PD), U5.9 (!PD), J32.1 (Pin_1)
- net +5V: now also J34.1 (Pin_1)
- net 15V_2: now also J36.1 (Pin_1)
- net 3v3_2: now also U12.9 (!PD), J33.1 (Pin_1)
- net Earth: now also J10.2 (Pin_2), J16.2 (Pin_2), J28.1 (Pin_1), J29.1 (Pin_1), J30.1 (Pin_1), J31.1 (Pin_1), J32.2 (Pin_2), J33.2 (Pin_2), J34.2 (Pin_2), J35.2 (Pin_2), J36.2 (Pin_2); no longer U12.9 (!PD), U20.9 (!PD), U5.9 (!PD)
- net at C68.1, H4.1 (Pin_1), J19.1 (Pin_1)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: now also R24.1; no longer R24.2
- net at C82.1, D12.2 (A), J15.1 (Pin_1)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: now also J16.1 (Pin_1)
- net at J4.3 (Pin_3), R9.2, U2.22 (TX2_io): now also J8.4 (Pin_4); no longer J8.3 (Pin_3)
- net at C81.1, D6.2 (A), J9.1 (Pin_1)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: now also J10.1 (Pin_1)
- net at J4.4 (Pin_4), R10.2, U2.13 (D13_a2io): now also J8.3 (Pin_3); no longer J8.4 (Pin_4)
- net at D7.1 (K), D8.1 (K), R16.1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: now also J27.1 (Pin_1)
- net at R22.2, U22.1 (G): now also R24.2; no longer R24.1
