File: Kicad/HVPSController2/_autosave-HVPSController2.kicad_pcb (KiCad board)
At the start: 4 copper layers, 314.1 x 184 mm, 178 parts, among them J1 Vsupply, J10 Tap debug pin, J11 USB RWGBS, J12 USB RWGBS, J13 Conn_01x01_Pin, J14 Conn_01x01_Pin, J15 Tap, J16 Tap debug pin, J17 Conn_01x02_Pin, J2 GND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

Commit message: Going great.
Parts:
- moved U25 9.69 mm to (218.5, 92.9)
- moved R29 4.50 mm to (216.8, 97.0)
- moved L2 0.85 mm to (203.7, 79.1)
Routing:
- net Net-(U25-G): track 97.8 -> 101.8 mm
- net Net-(D16-A): track 14.3 -> 12.8 mm
- net Net-(U2-D21_io): track 248.8 -> 247.7 mm
- net Net-(U3-IN+): track 12.9 -> 13.6 mm
Changed lines of the file:
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@@
 	(footprint "Resistor_THT:R_Axial_DIN0207_L6.3mm_D2.5mm_P7.62mm_Horizontal"
 		(layer "F.Cu")
-		(at 217.1 92.49 -90)
+		(at 216.8 96.98 -90)
 		(descr "Resistor, Axial_DIN0207 series, Axial, Horizontal, pin pitch=7.62mm, 0.25W = 1/4W, length*diameter=6.3*2.5mm^2, http://cdn-reichelt.de/documents/datenblatt/B400/1_4W%23YAG.pdf")
 		(tags "Resistor Axial_DIN0207 series Axial Horizontal pin pitch 7.62mm 0.25W = 1/4W length 6.3mm diameter 2.5mm")
@@
 	(footprint "Package_TO_SOT_THT:TO-92"
 		(layer "F.Cu")
-		(at 209.67 88.9 180)
+		(at 218.5 92.9 180)
 		(descr "TO-92 leads molded, narrow, drill 0.75mm (see NXP sot054_po.pdf)")
 		(tags "to-92 sc-43 sc-43a sot54 PA33 transistor")
@@
 	(footprint "Custom:5026 Inductor"
 		(layer "F.Cu")
-		(at 203.4 78.3 -90)
+		(at 203.7 79.1 -90)
 		(property "Reference" "L2"
 			(at 3 -6 -90)
@@
 	)
 	(segment
-		(start 207.3 78.3)
-		(end 203.4 78.3)
-		(width 2)
-		(layer "F.Cu")
-		(net 11)
-	)
-	(segment
 		(start 218.9 77.2)
 		(end 218.9 83.1)
@@
 	)
 	(segment
+		(start 208.7 76.9)
+		(end 206.5 79.1)
+		(width 2)
+		(layer "F.Cu")
+		(net 11)
+	)
+	(segment
 		(start 338.3 116.2)
 		(end 338.55 116.45)
@@
 	)
 	(segment
+		(start 206.5 79.1)
+		(end 203.7 79.1)
+		(width 2)
+		(layer "F.Cu")
+		(net 11)
+	)
+	(segment
+		(start 217.5 76.9)
+		(end 208.7 76.9)
+		(width 2)
+		(layer "F.Cu")
+		(net 11)
+	)
+	(segment
 		(start 253.56 199.3)
 		(end 249.55 199.3)
@@
 	)
 	(segment
-		(start 217.5 76.9)
-		(end 208.7 76.9)
-		(width 2)
-		(layer "F.Cu")
-		(net 11)
-	)
-	(segment
 		(start 73.9 241.5)
 		(end 80.8 248.4)
@@
 	)
 	(segment
-		(start 208.7 76.9)
-		(end 207.3 78.3)
-		(width 2)
-		(layer "F.Cu")
-		(net 11)
-	)
-	(segment
 		(start 218.5 76.8)
 		(end 218.9 77.2)
@@
 	)
 	(segment
-		(start 208.6 93.2)
-		(end 206.2 90.8)
+		(start 211.08 93.2)
+		(end 215.66 93.2)
 		(width 1)
 		(layer "F.Cu")
@@
 	)
 	(segment
-		(start 211.8 99.85)
-		(end 211.8 94.52)
+		(start 210.78 93.5)
+		(end 211.08 93.2)
 		(width 1)
 		(layer "F.Cu")
@@
 	)
 	(segment
-		(start 211.8 94.52)
-		(end 210.78 93.5)
+		(start 215.66 93.2)
+		(end 215.96 92.9)
 		(width 1)
 		(layer "F.Cu")
@@
 	)
 	(segment
-		(start 206.2 89.83)
-		(end 207.13 88.9)
+		(start 211.8 99.85)
+		(end 211.8 93.2)
 		(width 1)
 		(layer "F.Cu")
@@
 	)
 	(segment
-		(start 210.4 93.2)
-		(end 208.6 93.2)
+		(start 211.8 93.2)
+		(end 211.08 93.2)
 		(width 1)
 		(layer "F.Cu")
@@
 	)
 	(segment
-		(start 206.2 90.8)
-		(end 206.2 89.83)
-		(width 1)
-		(layer "F.Cu")
-		(net 51)
+		(start 210.57 90.67)
+		(end 214.3 94.4)
+		(width 0.5)
+		(layer "B.Cu")
+		(net 52)
+	)
+	(segment
+		(start 217.23 94.17)
+		(end 217.23 96.55)
+		(width 0.5)
+		(layer "B.Cu")
+		(net 52)
+	)
+	(segment
+		(start 214.3 94.4)
+		(end 217 94.4)
+		(width 0.5)
+		(layer "B.Cu")
+		(net 52)
+	)
+	(segment
+		(start 217 94.4)
+		(end 217.23 94.17)
+		(width 0.5)
+		(layer "B.Cu")
+		(net 52)
+	)
+	(segment
+		(start 217.23 96.55)
+		(end 216.8 96.98)
+		(width 0.5)
+		(layer "B.Cu")
+		(net 52)
 	)
 	(segment
 		(start 208.4 90.67)
-		(end 215.28 90.67)
+		(end 210.57 90.67)
 		(width 0.5)
 		(layer "B.Cu")
@@
 	)
 	(segment
-		(start 215.28 90.67)
-		(end 217.1 92.49)
-		(width 0.5)
-		(layer "B.Cu")
-		(net 52)
-	)
-	(segment
 		(start 218.8025 130.01375)
 		(end 214.8025 130.01375)
@@
 	)
 	(segment
-		(start 219.5 86.6)
-		(end 184 86.6)
-		(width 0.5)
-		(layer "B.Cu")
-		(net 161)
-	)
-	(segment
-		(start 294.19 95.2)
-		(end 291.29 92.3)
-		(width 0.5)
-		(layer "B.Cu")
-		(net 161)
-	)
-	(segment
-		(start 291.29 92.3)
-		(end 225.2 92.3)
+		(start 130.8 87.9)
+		(end 88.3 130.4)
 		(width 0.5)
 		(layer "B.Cu")
@@
 	)
 	(segment
-		(start 184 86.6)
-		(end 182.7 87.9)
+		(start 88.3 142.98)
+		(end 82.2 149.08)
 		(width 0.5)
 		(layer "B.Cu")
@@
 	)
 	(segment
-		(start 88.3 130.4)
-		(end 88.3 142.98)
+		(start 220.8 87.9)
+		(end 130.8 87.9)
 		(width 0.5)
 		(layer "B.Cu")
@@
 	(segment
 		(start 225.2 92.3)
-		(end 219.5 86.6)
+		(end 220.8 87.9)
 		(width 0.5)
 		(layer "B.Cu")
@@
 	)
 	(segment
-		(start 88.3 142.98)
-		(end 82.2 149.08)
+		(start 291.29 92.3)
+		(end 225.2 92.3)
 		(width 0.5)
 		(layer "B.Cu")
@@
 	)
 	(segment
-		(start 182.7 87.9)
-		(end 130.8 87.9)
+		(start 88.3 130.4)
+		(end 88.3 142.98)
 		(width 0.5)
 		(layer "B.Cu")
@@
 	)
 	(segment
-		(start 130.8 87.9)
-		(end 88.3 130.4)
+		(start 294.19 95.2)
+		(end 291.29 92.3)
 		(width 0.5)
 		(layer "B.Cu")
@@
 	)
 	(segment
-		(start 212.9 83.1)
-		(end 211.3 83.1)
+		(start 182.3 88.5)
+		(end 169.5 101.3)
 		(width 1)
 		(layer "F.Cu")
@@
 	)
 	(segment
-		(start 184.3 86.5)
-		(end 169.5 101.3)
+		(start 212.9 83.1)
+		(end 212.9 83.2)
 		(width 1)
 		(layer "F.Cu")
@@
 	)
 	(segment
-		(start 211.3 83.1)
-		(end 207.9 86.5)
+		(start 212.9 83.2)
+		(end 207.6 88.5)
 		(width 1)
 		(layer "F.Cu")
@@
 	)
 	(segment
-		(start 207.9 86.5)
-		(end 184.3 86.5)
+		(start 207.6 88.5)
+		(end 182.3 88.5)
 		(width 1)
 		(layer "F.Cu")
@@
 	)
 	(segment
-		(start 193.3 78.2)
-		(end 193.3 78.7)
+		(start 193.3 78.7)
+		(end 199.7 85.1)
 		(width 1)
 		(layer "F.Cu")
@@
 	)
 	(segment
-		(start 193.3 78.7)
-		(end 198.9 84.3)
+		(start 193.3 78.2)
+		(end 193.3 78.7)
 		(width 1)
 		(layer "F.Cu")
@@
 	)
 	(segment
-		(start 198.9 84.3)
-		(end 203.4 84.3)
+		(start 199.7 85.1)
+		(end 203.7 85.1)
 		(width 1)
 		(layer "F.Cu")
